File: example/arduino/Arduino FTDI UART.sch (EAGLE design)
At the start: 19 parts, among them IC1 FT232RL, X1 MINI-USB, X2 USB-A-SHIELD

Commit message: 2020.05.25.01
Parts:
- removed SV1: (no value), Pin-Header:MA08-1
- removed X2: USB-A-SHIELD, Socket:USB-A-SHIELD
- added SV2: (no value), Pin-Header:MA06-1
- X1: value MINI-USB -> MINI-USB-32005-201
Connections:
- removed net RX: IC1.RXD, R5.1, SV1.7
- removed net TX: IC1.TXD, R4.1, SV1.8
- new net N$2: IC1.TXD, R4.1
- new net N$8: IC1.RXD, R5.1
- net +3V3: now also SV2.5; no longer SV1.5
- net +5V: now also SV2.4; no longer SV1.4, X2.4
- net GND: now also SV2.1; no longer SV1.1, X2.1, X2.S1, X2.S2
- net RESET: now also SV2.6; no longer SV1.6
- net RXD: now also SV2.2; no longer SV1.3, X2.3
- net TXD: now also SV2.3; no longer SV1.2, X2.2
Other:
- moved on the sheet: 5V0LED, C1, C2, C4, D1, FUSE, IC1, R1, R2, R3, R4, R5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
