File: projects/Arduino Sersor Board/Arduino Sersor Board.brd (EAGLE design)
At the start: 68.6 x 53.3 mm, 45 parts, among them Q1 8050, Q2 S8050SOT23, X1 RELAY_OUT

Commit message: 2020.05.25.01
Parts:
- removed R10: 12k, RCLDA:R0805
- removed R9: 100, RCLDA:R0805
- turned LED4 to 270 degrees
Connections:
- removed net N$11: R9.2, U$9.VCC
- net +5V: now also U$9.VCC; no longer R10.1, R9.1
- net IR: no longer R10.2
Routing:
- net +5V: track 227.7 -> 233.4 mm
- net N$11: track 2.86 -> 0.00 mm
- net IR: track 48.9 -> 46.0 mm
- net DHT11: track 74.3 -> 76.8 mm
Changed lines of the file:
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@@
 <element name="R8" library="RCLDA" package="R0805" value="5K" x="22.86" y="16.51"/>
 <element name="U$9" library="Senser" package="IR-RECIEVER" value="IR-RECIEVER" x="63.5" y="19.05" rot="R90"/>
-<element name="R9" library="RCLDA" package="R0805" value="100" x="59.69" y="21.59" rot="MR180"/>
-<element name="R10" library="RCLDA" package="R0805" value="12k" x="59.69" y="16.51" rot="MR180"/>
 <element name="C1" library="RCLDA" package="C0805" value="104" x="59.69" y="19.05" rot="MR180"/>
 <element name="C2" library="RCLDA" package="C0805" value="104" x="22.86" y="13.97" rot="R180"/>
@@
 <element name="C4" library="RCLDA" package="C0805" value="104" x="22.225" y="3.81" rot="R270"/>
 <element name="R12" library="RCLDA" package="R0805" value="470" x="24.765" y="3.81" rot="R90"/>
-<element name="LED4" library="Display" package="CHIP-LED0805" value="RED" x="27.305" y="3.81" rot="R180"/>
+<element name="LED4" library="Display" package="CHIP-LED0805" value="RED" x="27.305" y="3.81" rot="R270"/>
 <element name="Q1" library="RCLDA" package="SOT23" value="8050" x="22.86" y="35.56" rot="MR90"/>
 <element name="C5" library="RCLDA" package="C0805" value="104" x="22.86" y="27.94" rot="MR90"/>
@@
 <contactref element="R2" pad="2"/>
 <contactref element="R8" pad="2"/>
-<contactref element="R9" pad="1"/>
-<contactref element="R10" pad="1"/>
-<contactref element="C1" pad="1"/>
 <contactref element="R4" pad="2"/>
 <contactref element="R5" pad="2"/>
@@
 <wire x1="54.61" y1="9.525" x2="54.61" y2="11.43" width="0.4064" layer="16"/>
 <contactref element="U$4" pad="1"/>
-<wire x1="58.74" y1="21.59" x2="58.74" y2="19.05" width="0.4064" layer="16"/>
-<wire x1="58.74" y1="19.05" x2="58.74" y2="16.51" width="0.4064" layer="16"/>
 <wire x1="55.56" y1="15.24" x2="55.56" y2="12.38" width="0.4064" layer="16"/>
 <wire x1="55.56" y1="12.38" x2="54.61" y2="11.43" width="0.4064" layer="16"/>
@@
 <wire x1="43.18" y1="11.43" x2="44.45" y2="10.16" width="0.4064" layer="1"/>
 <contactref element="U$1" pad="VCC"/>
-<wire x1="19.05" y1="12.7" x2="19.05" y2="13.97" width="0.4064" layer="1"/>
-<wire x1="58.74" y1="16.51" x2="56.83" y2="16.51" width="0.4064" layer="16"/>
-<wire x1="56.83" y1="16.51" x2="55.56" y2="15.24" width="0.4064" layer="16"/>
+<wire x1="19.05" y1="12.7" x2="17.78" y2="13.97" width="0.4064" layer="1"/>
 <wire x1="46.99" y1="43.18" x2="48.26" y2="43.18" width="0.4064" layer="1"/>
 <wire x1="48.26" y1="43.18" x2="49.53" y2="44.45" width="0.4064" layer="1"/>
@@
 <wire x1="55.245" y1="8.89" x2="54.61" y2="9.525" width="0.4064" layer="1"/>
 <wire x1="54.61" y1="9.525" x2="54.61" y2="11.43" width="0.4064" layer="1"/>
+<contactref element="U$9" pad="VCC"/>
+<contactref element="C1" pad="1"/>
+<wire x1="55.56" y1="15.24" x2="55.56" y2="18.73" width="0.4064" layer="16"/>
+<wire x1="55.56" y1="18.73" x2="55.88" y2="19.05" width="0.4064" layer="16"/>
+<wire x1="55.88" y1="19.05" x2="58.74" y2="19.05" width="0.4064" layer="16"/>
+<wire x1="58.74" y1="19.05" x2="58.74" y2="21.275" width="0.4064" layer="16"/>
+<wire x1="58.74" y1="21.275" x2="59.055" y2="21.59" width="0.4064" layer="16"/>
+<wire x1="59.055" y1="21.59" x2="63.5" y2="21.59" width="0.4064" layer="16"/>
 </signal>
 <signal name="GND">
@@
 <via x="26.67" y="16.51" extent="1-16" drill="0.5"/>
 <contactref element="U$1" pad="DAT"/>
-<wire x1="26.67" y1="16.51" x2="19.05" y2="16.51" width="0.4064" layer="16"/>
-<wire x1="19.05" y1="16.51" x2="21.91" y2="16.51" width="0.4064" layer="1"/>
+<wire x1="26.67" y1="16.51" x2="17.78" y2="16.51" width="0.4064" layer="16"/>
+<wire x1="17.78" y1="16.51" x2="21.91" y2="16.51" width="0.4064" layer="1"/>
 <wire x1="58.42" y1="50.8" x2="58.42" y2="48.895" width="0.4064" layer="16"/>
 <wire x1="58.42" y1="48.895" x2="57.785" y2="48.26" width="0.4064" layer="16"/>
@@
 <wire x1="48.895" y1="16.51" x2="26.67" y2="16.51" width="0.4064" layer="1"/>
 </signal>
-<signal name="N$11">
-<contactref element="R9" pad="2"/>
-<contactref element="U$9" pad="VCC"/>
-<wire x1="63.5" y1="21.59" x2="60.64" y2="21.59" width="0.4064" layer="16"/>
-</signal>
 <signal name="IR">
-<contactref element="R10" pad="2"/>
 <contactref element="U$9" pad="OUT"/>
 <contactref element="GND" pad="D4"/>
@@
 <wire x1="52.705" y1="17.145" x2="53.34" y2="16.51" width="0.4064" layer="1"/>
 <wire x1="53.34" y1="16.51" x2="63.5" y2="16.51" width="0.4064" layer="1"/>
-<wire x1="60.64" y1="16.51" x2="63.5" y2="16.51" width="0.4064" layer="16"/>
-</signal>
-<signal name="N$14">
-<contactref element="U$9" pad="GND"/>
-<contactref element="C1" pad="2"/>
-<wire x1="63.5" y1="19.05" x2="60.64" y2="19.05" width="0.4064" layer="16"/>
 </signal>
 <signal name="N$3">
@@
 <wire x1="48.26" y1="46.99" x2="46.99" y2="45.72" width="0.4064" layer="16"/>
 </signal>
+<signal name="N$8">
+<contactref element="U$9" pad="GND"/>
+<contactref element="C1" pad="2"/>
+<wire x1="60.64" y1="19.05" x2="63.5" y2="19.05" width="0.4064" layer="16"/>
+</signal>
 </signals>
