File: projects/Arduino Sersor Board/Arduino Sersor Board.sch (EAGLE design)
At the start: 45 parts, among them Q1 8050, Q2 S8050SOT23, X1 RELAY_OUT

Commit message: 2020.05.25.01
Parts:
- removed R10: 12k, RCLDA:RR0805
- removed R9: 100, RCLDA:RR0805
Connections:
- removed net N$11: R9.2, U$9.VCC
- net +5V: now also U$9.VCC; no longer R10.1, R9.1
- net IR: no longer R10.2
Other:
- moved on the sheet: C1
