File: projects/Arduino FTDI UART/Arduino FTDI UART.sch (EAGLE design)
At the start: 19 parts, among them IC1 FT232RL, X1 MINI-USB, X2 USB-A-SHIELD

Commit message: 2020.05.27.01
Parts:
- R1, R2: value 102 -> 331
- R3, R6: value 102 -> 471
Changed lines of the file:
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@@
 <setting verticaltext="up"/>
 </settings>
-<grid distance="50" unitdist="mil" unit="mil" style="lines" multiple="1" display="yes" altdistance="25" altunitdist="mil" altunit="mil"/>
+<grid distance="0.1" unitdist="inch" unit="inch" style="lines" multiple="1" display="no" altdistance="0.01" altunitdist="inch" altunit="inch"/>
 <layers>
 <layer number="1" name="Top" color="4" fill="1" visible="no" active="no"/>
@@
 <part name="VCCLED" library="Display" deviceset="LED" device="CHIPLED_0805" value="RED"/>
 <part name="C1" library="RCLDA" deviceset="C" device="C0805" value="104"/>
-<part name="R1" library="RCLDA" deviceset="R" device="R0805" value="102"/>
+<part name="R1" library="RCLDA" deviceset="R" device="R0805" value="331"/>
 <part name="D1" library="RCLDA" deviceset="DIODE" device="SMB"/>
 <part name="GND2" library="Power" deviceset="GND" device=""/>
@@
 <part name="FUSE" library="RCLDA" deviceset="R" device="R0805" value=""/>
 <part name="GND3" library="Power" deviceset="GND" device=""/>
-<part name="R2" library="RCLDA" deviceset="R" device="R0805" value="102"/>
+<part name="R2" library="RCLDA" deviceset="R" device="R0805" value="331"/>
 <part name="P+3" library="Power" deviceset="5V0" device=""/>
 <part name="P+4" library="Power" deviceset="5V0" device=""/>
-<part name="R3" library="RCLDA" deviceset="R" device="R0805" value="102"/>
+<part name="R3" library="RCLDA" deviceset="R" device="R0805" value="471"/>
 <part name="GND4" library="Power" deviceset="GND" device=""/>
 <part name="C2" library="RCLDA" deviceset="C" device="C0805" value="104"/>
@@
 <part name="R5" library="RCLDA" deviceset="R" device="R0805" value="102"/>
 <part name="P+9" library="Power" deviceset="5V0" device=""/>
-<part name="R6" library="RCLDA" deviceset="R" device="R0805" value="102"/>
+<part name="R6" library="RCLDA" deviceset="R" device="R0805" value="471"/>
 <part name="5V0LED" library="Display" deviceset="LED" device="CHIPLED_0805" value="RED"/>
 <part name="GND8" library="Power" deviceset="GND" device=""/>

Commit message: 2020.06.01.01
Parts:
- removed FUSE: RR0805, RCLDA:RR0805
- added U$1: FUSE0805, RCLDA:FUSE0805
Connections:
- net DM: now also X1.2; no longer X1.4
- net GND: now also X1.5; no longer X1.1
- net N$3: now also U$1.P$1, X1.1; no longer FUSE.1, X1.5
- net VCC: now also U$1.P$2; no longer FUSE.2
Other:
- moved on the sheet: D1, R3, VCCLED, X1
