File: projects/Arduino Emoji/Arduino Emoji.brd (EAGLE design)
At the start: 240.7 x 59.7 mm, 34 parts, among them M1 MAX7219, M2 MAX7219, M3 MAX7219, M4 MAX7219, Y1 16MHZ

Commit message: 2020.06.05.01
Parts:
- removed DIODE: 1N4007, RCLDA:RDIP
- removed EC1: 47u, RCLDA:ELECTRO-DIP
- removed L1, L3, L4: DOT-MATRIX-BS2088BS, Display:2088BS
- removed M1, M3, M4: MAX7219, Chip:SOP24
- removed R5, R7, R8: RDIP, RCLDA:RDIP
- removed SV2: (no value), Pin-Header:MA03-2
- added CT1: 100UF, RCLDA:ELECTRO-SMD-C-6.0MM
- added D1: DIODESMB, RCLDA:SMB
- added IN, OUT: (no value), Pin-Header:MA06-1
- C1, C3, C4, C5, C6: device RCLDA:CDIP -> RCLDA:C0805
- LED1, LED2, LED3: device Display:LED2X5 -> Display:CHIPLED_0805
- R1, R2, R3, R4: device RCLDA:RDIP -> RCLDA:R0805
- R6: value RDIP -> R0805; device RCLDA:RDIP -> RCLDA:R0805
- moved R6 112.0 mm to (41.3, 18.4), flipped to the bottom, turned to 180 degrees
- moved C4 90.0 mm to (41.3, 36.2), flipped to the bottom, turned to 180 degrees
- moved SJ1 88.3 mm to (33.3, 31.1), turned to 180 degrees
- moved C3 85.0 mm to (41.3, 33.7), flipped to the bottom, turned to 180 degrees
- moved U1 82.9 mm to (37.5, 29.8), turned to 90 degrees
- moved R4 81.2 mm to (33.7, 36.2), flipped to the bottom, turned to 0 degrees
- moved LED3 77.6 mm to (33.7, 38.7), flipped to the bottom, turned to 0 degrees
- moved Y1 77.2 mm to (50.2, 34.9), turned to 270 degrees
- moved M2 73.0 mm to (17.1, 29.8), turned to 90 degrees
- moved SV1 69.6 mm to (50.8, 2.54), turned to 180 degrees
- moved S1 67.5 mm to (55.2, 10.2), turned to 90 degrees
- moved C1 62.8 mm to (41.3, 13.3), flipped to the bottom, turned to 0 degrees
- moved R2 62.8 mm to (41.3, 15.9), flipped to the bottom, turned to 180 degrees
- moved L2 60.3 mm to (29.8, 29.8)
- moved LED1 10.6 mm to (9.53, 17.8)
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Connections:
- net N$11 renamed R6
- net N$12 renamed R7
- net N$13 renamed R8
- net N$30 renamed R1
- net N$31 renamed C1
- net N$32 renamed C2
- net N$33 renamed C3
- net N$34 renamed C4
- net N$35 renamed C5
- net N$36 renamed C6
- net N$37 renamed C7
- net N$38 renamed C8
- net N$5 renamed R2
- net N$7 renamed R3
- net N$8 renamed R4
- net N$9 renamed R5
- removed net N$14: L1.ROW1, M1.22
- removed net N$15: L1.ROW8, M1.17
- removed net N$16: L1.ROW7, M1.15
- removed net N$17: L1.ROW6, M1.21
- removed net N$18: L1.ROW5, M1.23
- removed net N$19: L1.ROW4, M1.20
- removed net N$20: L1.ROW3, M1.16
- removed net N$21: L1.ROW2, M1.14
- removed net N$22: L1.COL1, M1.2
- removed net N$23: L1.COL2, M1.11
- removed net N$24: L1.COL3, M1.6
- removed net N$25: L1.COL4, M1.7
- removed net N$26: L1.COL5, M1.3
- removed net N$27: L1.COL6, M1.10
- removed net N$28: L1.COL7, M1.5
- removed net N$29: L1.COL8, M1.8
- removed net N$39: L4.ROW2, M4.14
- removed net N$40: M2.18, R6.P$2
- removed net N$41: L4.ROW3, M4.16
- removed net N$42: L4.ROW4, M4.20
- removed net N$43: L4.ROW5, M4.23
- removed net N$44: L4.ROW6, M4.21
- removed net N$45: L4.ROW7, M4.15
- removed net N$46: L4.ROW8, M4.17
- removed net N$47: L4.ROW1, M4.22
- removed net N$48: L4.COL1, M4.2
- removed net N$49: L4.COL2, M4.11
- removed net N$50: L4.COL3, M4.6
- removed net N$51: L4.COL4, M4.7
- removed net N$52: L4.COL5, M4.3
- removed net N$53: L4.COL6, M4.10
- removed net N$54: L4.COL7, M4.5
- removed net N$55: L4.COL8, M4.8
- removed net N$56: L3.ROW2, M3.14
- removed net N$57: L3.ROW3, M3.16
- removed net N$58: L3.ROW4, M3.20
- removed net N$59: L3.ROW5, M3.23
- removed net N$60: L3.ROW6, M3.21
- removed net N$61: L3.ROW7, M3.15
- removed net N$62: M4.18, R7.P$2
- removed net N$63: L3.ROW8, M3.17
- removed net N$64: L3.ROW1, M3.22
- removed net N$65: L3.COL1, M3.2
- removed net N$66: L3.COL2, M3.11
- removed net N$67: L3.COL3, M3.6
- removed net N$68: L3.COL4, M3.7
- removed net N$69: L3.COL5, M3.3
- removed net N$70: L3.COL6, M3.10
- removed net N$71: L3.COL7, M3.5
- removed net N$72: L3.COL8, M3.8
- removed net N$73: M3.18, R8.P$2
- removed net N$74: M1.24, M2.1
- removed net N$75: M2.24, M3.1
- removed net N$76: M3.24, M4.1
- new net DOUT: IN.2, M2.24, OUT.3
- net +5V: now also C6.2, D1.1, IN.6, OUT.6, R1.2, R2.1, R3.2, R6.1; no longer C6.P$2, DIODE.P$2, M1.19, M3.19, M4.19, R1.P$2, R2.P$1, R3.P$2, R5.P$1, R6.P$1, R7.P$1, R8.P$1, SV2.5
- net CLK: now also IN.4, OUT.4; no longer M1.13, M3.13, M4.13
- net CS: now also IN.5, OUT.5; no longer M1.12, M3.12, M4.12
- net DIN: now also IN.3, M2.1, OUT.2; no longer M1.1
- net GND: now also C3.1, C4.1, C5.2, C6.1, CT1.-, IN.1, LED1.C, LED2.C, LED3.C, OUT.1; no longer C3.P$1, C4.P$1, C5.P$2, C6.P$1, EC1.-, LED1.K, LED2.K, LED3.K, M1.4, M1.9, M3.4, M3.9, M4.4, M4.9, SV2.1
- net MISO: no longer SV2.6
- net MOSI: no longer SV2.3
- net N$1: now also R4.1; no longer R4.P$1
- net N$10: now also R3.1; no longer R3.P$1
- net N$2: now also D1.2; no longer DIODE.P$1
- net N$3: now also C1.2; no longer C1.P$2
- net N$4: now also R1.1; no longer R1.P$1
- net N$6: now also M2.18, R6.2; no longer M1.18, R5.P$2
- net RST: now also C1.1, R2.2; no longer C1.P$1, R2.P$2, SV2.2
- net SCK: now also R4.2; no longer R4.P$2, SV2.4
- net VCC: now also C5.1, CT1.+; no longer C5.P$1, EC1.+
- net X1: now also C3.2; no longer C3.P$2
- net X2: now also C4.2; no longer C4.P$2
Routing:
- net R3: track 0.00 -> 67.8 mm, vias 0 -> 2
- net +5V: track 0.00 -> 50.5 mm, vias 0 -> 2
- net R8: track 0.00 -> 49.1 mm, vias 0 -> 1
- net C4: track 0.00 -> 47.9 mm, vias 0 -> 3
- net R6: track 0.00 -> 46.7 mm, vias 0 -> 2
- net R2: track 0.00 -> 39.2 mm
- net C1: track 0.00 -> 35.1 mm
- net C6: track 0.00 -> 35.1 mm, vias 0 -> 4
- net R1: track 0.00 -> 35.1 mm
- net DOUT: track 0.00 -> 33.9 mm
- net R7: track 0.00 -> 33.1 mm
- net C3: track 0.00 -> 32.4 mm
- net C7: track 0.00 -> 31.8 mm
- net C5: track 0.00 -> 29.5 mm
- net C8: track 0.00 -> 27.7 mm
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Other:
- board size 240.7 x 59.7 mm -> 59.7 x 59.7 mm
