File: projects/Arduino Emoji/Arduino Emoji.sch (EAGLE design)
At the start: 34 parts, among them M1 MAX7219, M2 MAX7219, M3 MAX7219, M4 MAX7219, Y1 16MHZ

Commit message: 2020.06.05.01
Parts:
- removed DIODE: 1N4007, RCLDA:RDIP
- removed EC1: 47u, RCLDA:ELECTRO-DIP
- removed L1, L3, L4: DOT-MATRIX-BS2088BS, Display:DOT-MATRIX-BS2088BS
- removed M1, M3, M4: MAX7219, Chip:MAX7219
- removed R5, R7, R8: RDIP, RCLDA:RDIP
- removed SV2: (no value), Pin-Header:MA03-2
- added CT1: 100UF, RCLDA:ALUMINUM-SMD-100UF-50V(D6.0-H6.0MM)
- added D1: DIODESMB, RCLDA:DIODESMB
- added IN, OUT: (no value), Pin-Header:MA06-1
- C1, C3, C4, C5, C6: device RCLDA:CDIP -> RCLDA:C0805
- LED1, LED2, LED3: device Display:LEDSQR2X5 -> Display:LEDCHIPLED_0805
- R1, R2, R3, R4: device RCLDA:RDIP -> RCLDA:R0805
- R6: value RDIP -> R0805; device RCLDA:RDIP -> RCLDA:R0805
Connections:
- net N$11 renamed R6
- net N$12 renamed R7
- net N$13 renamed R8
- net N$30 renamed R1
- net N$31 renamed C1
- net N$32 renamed C2
- net N$33 renamed C3
- net N$34 renamed C4
- net N$35 renamed C5
- net N$36 renamed C6
- net N$37 renamed C7
- net N$38 renamed C8
- net N$5 renamed R2
- net N$7 renamed R3
- net N$8 renamed R4
- net N$9 renamed R5
- removed net N$14: L1.ROW1, M1.SEGH
- removed net N$15: L1.ROW8, M1.SEGG
- removed net N$16: L1.ROW7, M1.SEGF
- removed net N$17: L1.ROW6, M1.SEGE
- removed net N$18: L1.ROW5, M1.SEGD
- removed net N$19: L1.ROW4, M1.SEGC
- removed net N$20: L1.ROW3, M1.SEGB
- removed net N$21: L1.ROW2, M1.SEGA
- removed net N$22: L1.COL1, M1.DIG0
- removed net N$23: L1.COL2, M1.DIG1
- removed net N$24: L1.COL3, M1.DIG2
- removed net N$25: L1.COL4, M1.DIG3
- removed net N$26: L1.COL5, M1.DIG4
- removed net N$27: L1.COL6, M1.DIG5
- removed net N$28: L1.COL7, M1.DIG6
- removed net N$29: L1.COL8, M1.DIG7
- removed net N$39: L4.ROW2, M4.SEGA
- removed net N$41: L4.ROW3, M4.SEGB
- removed net N$42: L4.ROW4, M4.SEGC
- removed net N$43: L4.ROW5, M4.SEGD
- removed net N$44: L4.ROW6, M4.SEGE
- removed net N$45: L4.ROW7, M4.SEGF
- removed net N$46: L4.ROW8, M4.SEGG
- removed net N$47: L4.ROW1, M4.SEGH
- removed net N$48: L4.COL1, M4.DIG0
- removed net N$49: L4.COL2, M4.DIG1
- removed net N$50: L4.COL3, M4.DIG2
- removed net N$51: L4.COL4, M4.DIG3
- removed net N$52: L4.COL5, M4.DIG4
- removed net N$53: L4.COL6, M4.DIG5
- removed net N$54: L4.COL7, M4.DIG6
- removed net N$55: L4.COL8, M4.DIG7
- removed net N$56: L3.ROW2, M3.SEGA
- removed net N$57: L3.ROW3, M3.SEGB
- removed net N$58: L3.ROW4, M3.SEGC
- removed net N$59: L3.ROW5, M3.SEGD
- removed net N$6 (its old number): M1.ISET, R5.2
- removed net N$60: L3.ROW6, M3.SEGE
- removed net N$61: L3.ROW7, M3.SEGF
- removed net N$62: M4.ISET, R7.2
- removed net N$63: L3.ROW8, M3.SEGG
- removed net N$64: L3.ROW1, M3.SEGH
- removed net N$65: L3.COL1, M3.DIG0
- removed net N$66: L3.COL2, M3.DIG1
- removed net N$67: L3.COL3, M3.DIG2
- removed net N$68: L3.COL4, M3.DIG3
- removed net N$69: L3.COL5, M3.DIG4
- removed net N$70: L3.COL6, M3.DIG5
- removed net N$71: L3.COL7, M3.DIG6
- removed net N$72: L3.COL8, M3.DIG7
- removed net N$73: M3.ISET, R8.2
- removed net N$74: M1.DOUT, M2.DIN
- removed net N$75: M2.DOUT, M3.DIN
- removed net N$76: M3.DOUT, M4.DIN
- new net DOUT: IN.2, M2.DOUT, OUT.3
- net +5V: now also D1.1, IN.6, OUT.6; no longer DIODE.2, M1.VCC, M3.VCC, M4.VCC, R5.1, R7.1, R8.1, SV2.5
- net CLK: now also IN.4, OUT.4; no longer M1.CLK, M3.CLK, M4.CLK
- net CS: now also IN.5, OUT.5; no longer M1.CS, M3.CS, M4.CS
- net DIN: now also IN.3, M2.DIN, OUT.2; no longer M1.DIN
- net GND: now also CT1.-, IN.1, OUT.1; no longer EC1.-, M1.GND, M1.VSS, M3.GND, M3.VSS, M4.GND, M4.VSS, SV2.1
- net MISO: no longer SV2.6
- net MOSI: no longer SV2.3
- net N$2: now also D1.2; no longer DIODE.1
- net RST: no longer SV2.2
- net SCK: no longer SV2.4
- net VCC: now also CT1.+; no longer EC1.+
