File: projects/Arduino Basic Sensor Board/Arduino Basic Sensor Board.sch (EAGLE design)
At the start: 35 parts, among them Q1 S8050SOT23, Q2 S8050SOT23, U1 74HC595N-DIP16

Commit message: 2020.06.08.01
Parts:
- removed LED3: GREEN, Display:LEDSQR2X5
- removed U1: 74HC595N-DIP16, Chip:LOGIC-74HC595N(DIP16)
- added JP1, JP2: (no value), Jumper:JP1Q
- added LED10: RED, Display:LEDSML1206
- added LED11: YELLOW, Display:LEDSML1206
- added LED12: GREEN, Display:LEDSML1206
- added R12, R13, R14: 103, RCLDA:R0805
- added S3: TS-SMD_6S6_SHIELD, Button:TS-SMD_6S6_SHIELD
- added SV4, SV5: (no value), Pin-Header:MA03-1
- added U$15: 3261AS, Display:3261AS
- LED1: value RED -> (none); device Display:LEDSQR2X5 -> Display:LEDCHIPLED_1206
- LED2: value YELLOW -> (none); device Display:LEDSQR2X5 -> Display:LEDCHIPLED_1206
- SV1: device Pin-Header:MA04-1 -> Pin-Header:MA03-1
- U$8: value LG3622BH -> TM1650; device Display:LG3622BH -> Chip:TM1650
Connections:
- removed net A4: U$1.A4/SDA
- removed net A5: U$1.A5/SCL
- new net DIG1: U$15.DIG1, U$8.DIG1
- new net DIG2: U$15.DIG2, U$8.DIG2
- new net N$12: LED2.A, R14.1
- new net N$13: JP1.2, JP2.2, SV2.2
- new net N$7: LED1.A, R13.1
- net 3V3: now also JP2.1
- net 5V0: now also JP1.1, R12.1, SV1.2, SV4.2, SV5.2, U$8.VDD; no longer SV1.4, SV2.4, U1.!MR, U1.VCC
- net A: now also U$15.A; no longer U1.Q0
- net B: now also U$15.B; no longer U1.Q1
- net C: now also U$15.C; no longer U1.Q2
- net D: now also U$15.D; no longer U1.Q3
- net D11: now also LED12.C; no longer LED3.C
- net D12: now also LED11.C; no longer LED2.C
- net D13: now also LED10.C; no longer LED1.C
- net D2: now also SV5.3; no longer U$8.2
- net D3: now also SV4.3; no longer U$8.1
- net D4: now also SV1.3; no longer U1.STCP
- net D5: now also R14.2; no longer U1.SHCP
- net D6: now also R13.2; no longer U1.DS
- net D7: now also R8.1; no longer R9.2, U$4.DAT
- net D8: now also R9.2, U$4.DAT; no longer R8.1
- net E: now also U$15.E; no longer U1.Q4
- net F: now also U$15.F; no longer U1.Q5
- net G: now also U$15.G; no longer U1.Q6
- net GND: now also LED1.C, LED2.C, S3.1.1, S3.1.2, S3.SH, SV4.1, SV5.1, U$8.GND; no longer U1.!OE, U1.GND
- net H: now also U$15.DP; no longer U1.Q7
- net N$1: now also LED10.A; no longer LED1.A
- net N$2: now also LED11.A; no longer LED2.A
- net N$3: now also LED12.A; no longer LED3.A
- net RESET: now also R12.2, S3.2.1, S3.2.2
- net RXD: now also SV2.4; no longer SV2.2
- net SCL: now also U$1.A5/SCL, U$8.SCL; no longer SV1.3, U$1.SCL
- net SDA: now also U$1.A4/SDA, U$8.SDA; no longer SV1.2, U$1.SDA
Other:
- note added: "DIGITAL(D4/D3/D2)"
- note added: "DISPLAY(A4/A5)"
- note added: "PWM(D6/D5)"
- note added: "RESET"
- note removed: "74HC595(D6/D5/D4/D3/D2)"
- note removed: "IIC(A4/A5)"
- moved on the sheet: LED1, LED2, R5, SV2, SV3, U$2, U$5, U$6
