File: projects/03 Arduino Advanced Sensor Board/Arduino Advanced Sensor Board.brd (EAGLE design)
At the start: 18.1 x 1 mm, 34 parts

Commit message: 2020.06.16.01
Parts:
- added R10, R11, R9: 102, RCLDA:R0805
- added R12, R13, R14: 222, RCLDA:R0805
- moved U$5 37.5 mm to (54.6, 8.89)
- moved U$2 36.1 mm to (54.6, 8.89), turned to 180 degrees
- moved G1 35.5 mm to (38.1, 12.1), turned to 90 degrees
- moved SD1 0.63 mm to (14.0, 35.6)
Connections:
- removed net A0: U$1.A0
- removed net A1: U$1.A1
- removed net A2: U$1.A2
- removed net D2: U$1.D2
- removed net D3: U$1.D3
- removed net D4: U$1.D4
- new net MISO: SD1.7, U$1.D12
- new net MOSI: R10.1, U$1.D11
- new net N$10: R10.2, R13.1, SD1.3
- new net N$12: R12.1, R9.2, SD1.5
- new net N$9: R11.2, R14.1, SD1.2
- new net SCK: R9.1, U$1.D13
- new net SS: R11.1, U$1.D10
- net 3V3: now also SD1.4
- net CE: now also U$1.A0; no longer U$1.D5
- net GND: now also R12.2, R13.2, R14.2, SD1.6, SD1.G1, SD1.G2, SD1.G3, SD1.G4
- net IN1: now also U$1.D2; no longer U$1.D13
- net IN2: now also U$1.D3; no longer U$1.D12
- net IN3: now also U$1.D4; no longer U$1.D9
- net IN4: now also U$1.D7; no longer U$1.D8
- net IO: now also U$1.A1; no longer U$1.D6
- net PWM1: now also U$1.D5; no longer U$1.D11
- net PWM2: now also U$1.D6; no longer U$1.D10
- net SCLK: now also U$1.A2; no longer U$1.D7
Routing:
- net SDA: track 44.7 -> 0.00 mm, vias 1 -> 0
- net SCL: track 39.3 -> 0.00 mm
- net OUT3: track 35.6 -> 0.00 mm
- net OUT4: track 26.6 -> 0.00 mm
- net 3V3: track 26.0 -> 0.00 mm
- net VIN: track 24.3 -> 0.00 mm
- net OUT1: track 21.3 -> 0.00 mm
- net RES: track 14.7 -> 0.00 mm
- net C1N: track 14.6 -> 0.00 mm
- net C1P: track 13.8 -> 0.00 mm
- net TXD: track 11.1 -> 0.00 mm
- net IREF: track 10.3 -> 0.00 mm
- net VDD: track 9.52 -> 0.00 mm
- net C2N: track 9.21 -> 0.00 mm
- net D/C: track 8.96 -> 0.00 mm
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