File: projects/03 Arduino Advanced Sensor Board/Arduino Advanced Sensor Board.brd (EAGLE design)
At the start: 68.6 x 53.3 mm, 44 parts

Commit message: 2020.06.19.01
Parts:
- added U$17: (no value), Logos:MAKE_SOMETHING_FUN_100
- moved FUSE 6.70 mm to (21.0, 7.30), turned to 0 degrees
- moved R1 1.27 mm to (14.3, 3.81), turned to 0 degrees
- moved U$5 0.95 mm to (54.6, 9.84)
- moved U$13 0.64 mm to (21.6, 42.5)
- moved U$16 0.64 mm to (21.6, 37.5)
- moved U$14 0.63 mm to (21.6, 39.4)
- moved U$15 0.63 mm to (32.4, 42.9)
Routing:
- net 3V3: track 0.00 -> 150.6 mm, vias 0 -> 1
- net 5V0: track 0.00 -> 119.6 mm
- net IN1: track 0.00 -> 62.4 mm, vias 0 -> 1
- net IN4: track 0.00 -> 61.8 mm
- net IN3: track 0.00 -> 58.6 mm, vias 0 -> 1
- net PWM1: track 0.00 -> 56.6 mm
- net PWM2: track 0.00 -> 52.1 mm, vias 0 -> 1
- net IN2: track 0.00 -> 49.1 mm, vias 0 -> 1
- net SDA: track 0.00 -> 43.1 mm, vias 0 -> 1
- net SCL: track 0.00 -> 38.8 mm
- net RESET: track 0.00 -> 37.3 mm, vias 0 -> 1
- net OUT2: track 0.00 -> 34.1 mm
- net VCC: track 0.00 -> 28.1 mm
- net VIN: track 0.00 -> 26.9 mm
- net N$6: track 0.00 -> 24.1 mm
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
Commit message: 2020.06.26.01
Parts:
- added SV3, SV4: (no value), Pin-Header:MA03-1
- added U$18: (no value), Logos:D8_050
- added U$19: (no value), Logos:D9_050
- added U$20: (no value), Logos:5V0_050
- added U$21: (no value), Logos:GND_050
- U$13: device Logos:LOGO_100 -> Logos:ARDUINO_ADVANCED_SENSOR_BOARD
- U$14: device Logos:WWW.DIOSTUDIO.CN_100 -> Logos:DIOSTUDIO_100
- U$15: device Logos:DIOSTUDIO_100 -> Logos:LOGO_100
- U$16: device Logos:ARDUINO_ADVANCED_SENSOR_BOARD -> Logos:WWW.DIOSTUDIO.CN_100
- moved U$14 11.2 mm to (32.4, 42.2)
- moved U$15 10.8 mm to (21.6, 41.9)
- moved U$13 5.72 mm to (21.6, 36.8)
- moved U$16 1.27 mm to (21.6, 38.7)
- moved U$17 0.64 mm to (52.1, 36.8)
Connections:
- new net D8: SV3.3, U$1.D8
- new net D9: SV4.3, U$1.D9
- net 5V0: now also SV3.2, SV4.2
- net GND: now also SV3.1, SV4.1
Routing:
- net 5V0: track 119.6 -> 158.0 mm
- net D8: track 0.00 -> 30.1 mm
- net D9: track 0.00 -> 29.4 mm
- net OUT2: track 34.1 -> 28.7 mm
- net PWM1: track 56.6 -> 61.1 mm, vias 0 -> 1
- net IN2: track 49.1 -> 51.7 mm, vias 1 -> 0
- net IN1: track 62.4 -> 64.9 mm
- net OUT1: track 23.2 -> 21.4 mm
- net IN4: track 61.8 -> 63.5 mm, vias 0 -> 1
- net IN3: track 58.6 -> 59.2 mm, vias 1 -> 0
- net 3V3: track 150.6 -> 150.7 mm, vias 1 -> 2
- net PWM2: vias 1 -> 0
Other:
- board text added: "1"
- board text added: "30"
- board text added: "JLCJLCJLCJLC"

Commit message: 2020.06.30.01
Parts:
- added SV2: (no value), Pin-Header:MA03-1
- added U$22: (no value), Logos:A3_050
- moved U$20 8.89 mm to (22.2, 23.5)
- moved U$21 8.89 mm to (22.2, 21.0)
- moved U$17 0.32 mm to (52.1, 37.1)
Connections:
- net 5V0: now also SV2.2
- net A3: now also SV2.3
- net GND: now also SV2.1
Routing:
- net A3: track 0.00 -> 65.2 mm, vias 0 -> 3
- net 5V0: track 158.0 -> 157.3 mm
Changed lines of the file:
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@@
 <element name="U$15" library="Logos" package="LOGO_100" value="" x="21.59" y="41.91"/>
 <element name="U$16" library="Logos" package="WWW.DIOSTUDIO.CN_100" value="" x="21.59" y="38.735"/>
-<element name="U$17" library="Logos" package="MAKE_SOMETHING_FUN_100" value="" x="52.07" y="36.83" rot="MR0"/>
+<element name="U$17" library="Logos" package="MAKE_SOMETHING_FUN_100" value="" x="52.07" y="37.1475" rot="MR0"/>
 <element name="U$18" library="Logos" package="D8_050" value="" x="28.575" y="28.575"/>
 <element name="U$19" library="Logos" package="D9_050" value="" x="26.035" y="28.575"/>
-<element name="U$20" library="Logos" package="5V0_050" value="" x="31.115" y="23.495"/>
-<element name="U$21" library="Logos" package="GND_050" value="" x="31.115" y="20.955"/>
+<element name="U$20" library="Logos" package="5V0_050" value="" x="22.225" y="23.495"/>
+<element name="U$21" library="Logos" package="GND_050" value="" x="22.225" y="20.955"/>
+<element name="SV2" library="Pin-Header" package="MA03-1" value="" x="31.75" y="24.13" rot="R90">
+<attribute name="MPN" value="" x="31.75" y="24.13" size="1.778" layer="27" rot="R90" display="off"/>
+<attribute name="OC_NEWARK" value="unknown" x="31.75" y="24.13" size="1.778" layer="27" rot="R90" display="off"/>
+<attribute name="MF" value="" x="31.75" y="24.13" size="1.778" layer="27" rot="R90" display="off"/>
+<attribute name="OC_FARNELL" value="unknown" x="31.75" y="24.13" size="1.778" layer="27" rot="R90" display="off"/>
+</element>
+<element name="U$22" library="Logos" package="A3_050" value="" x="31.115" y="28.575"/>
 </elements>
 <signals>
@@
 <wire x1="53.975" y1="44.45" x2="53.975" y2="42.545" width="0.6096" layer="1"/>
 <wire x1="26.67" y1="24.13" x2="29.21" y2="24.13" width="0.6096" layer="1"/>
-<wire x1="29.21" y1="24.13" x2="30.48" y2="24.13" width="0.6096" layer="1"/>
-<wire x1="30.48" y1="24.13" x2="31.4325" y2="25.0825" width="0.6096" layer="1"/>
-<wire x1="31.4325" y1="25.0825" x2="31.4325" y2="31.75" width="0.6096" layer="1"/>
-<wire x1="31.4325" y1="31.75" x2="32.0675" y2="32.385" width="0.6096" layer="1"/>
-<wire x1="32.0675" y1="32.385" x2="38.1" y2="32.385" width="0.6096" layer="1"/>
-<wire x1="38.1" y1="32.385" x2="48.26" y2="42.545" width="0.6096" layer="1"/>
+<wire x1="35.8775" y1="30.1625" x2="48.26" y2="42.545" width="0.6096" layer="1"/>
 <wire x1="48.26" y1="42.545" x2="53.975" y2="42.545" width="0.6096" layer="1"/>
+<contactref element="SV2" pad="2"/>
+<wire x1="29.21" y1="24.13" x2="31.75" y2="24.13" width="0.6096" layer="1"/>
+<wire x1="31.75" y1="24.13" x2="35.2425" y2="24.13" width="0.6096" layer="1"/>
+<wire x1="35.2425" y1="24.13" x2="35.8775" y2="24.765" width="0.6096" layer="1"/>
+<wire x1="35.8775" y1="24.765" x2="35.8775" y2="30.1625" width="0.6096" layer="1"/>
 </signal>
 <signal name="GND">
@@
 <contactref element="SV3" pad="1"/>
 <contactref element="SV4" pad="1"/>
+<contactref element="SV2" pad="1"/>
 </signal>
 <signal name="A3">
 <contactref element="U$1" pad="A3"/>
+<contactref element="SV2" pad="3"/>
+<wire x1="58.42" y1="2.54" x2="62.23" y2="6.35" width="0.3048" layer="1"/>
+<wire x1="62.23" y1="6.35" x2="66.675" y2="6.35" width="0.3048" layer="1"/>
+<wire x1="66.675" y1="6.35" x2="67.31" y2="6.985" width="0.3048" layer="1"/>
+<wire x1="67.31" y1="6.985" x2="67.31" y2="19.685" width="0.3048" layer="1"/>
+<via x="67.31" y="19.685" extent="1-16" drill="0.5"/>
+<wire x1="67.31" y1="19.685" x2="67.31" y2="20.32" width="0.3048" layer="16"/>
+<wire x1="67.31" y1="20.32" x2="66.9925" y2="20.6375" width="0.3048" layer="16"/>
+<wire x1="66.9925" y1="20.6375" x2="59.055" y2="20.6375" width="0.3048" layer="16"/>
+<via x="59.055" y="20.6375" extent="1-16" drill="0.5"/>
+<wire x1="59.055" y1="20.6375" x2="34.6075" y2="20.6375" width="0.3048" layer="1"/>
+<wire x1="34.6075" y1="20.6375" x2="34.29" y2="20.955" width="0.3048" layer="1"/>
+<wire x1="34.29" y1="20.955" x2="34.29" y2="22.5425" width="0.3048" layer="1"/>
+<via x="34.29" y="22.5425" extent="1-16" drill="0.5"/>
+<wire x1="34.29" y1="22.5425" x2="34.29" y2="26.035" width="0.3048" layer="16"/>
+<wire x1="34.29" y1="26.035" x2="33.655" y2="26.67" width="0.3048" layer="16"/>
+<wire x1="33.655" y1="26.67" x2="31.75" y2="26.67" width="0.3048" layer="16"/>
 </signal>
 <signal name="SDA">
@@
 <wire x1="66.3575" y1="6.0325" x2="65.405" y2="5.08" width="0.3048" layer="16"/>
 <via x="65.405" y="5.08" extent="1-16" drill="0.5"/>
-<wire x1="65.405" y1="5.08" x2="61.595" y2="5.08" width="0.3048" layer="1"/>
-<wire x1="61.595" y1="5.08" x2="60.96" y2="4.445" width="0.3048" layer="1"/>
-<wire x1="60.96" y1="4.445" x2="60.96" y2="2.54" width="0.3048" layer="1"/>
+<wire x1="65.405" y1="5.08" x2="62.23" y2="5.08" width="0.3048" layer="1"/>
+<wire x1="62.23" y1="5.08" x2="60.96" y2="3.81" width="0.3048" layer="1"/>
+<wire x1="60.96" y1="3.81" x2="60.96" y2="2.54" width="0.3048" layer="1"/>
 </signal>
 <signal name="SCL">

Commit message: 2020.07.01.01
Parts:
- removed SV2, SV3, SV4: (no value), Pin-Header:MA03-1
- removed U$18: (no value), Logos:D8_050
- removed U$19: (no value), Logos:D9_050
- removed U$20: (no value), Logos:5V0_050
- removed U$21: (no value), Logos:GND_050
- removed U$22: (no value), Logos:A3_050
- added U$23, U$24, U$25: (no value), Button:TS-SMD_3*6
- U$14: device Logos:DIOSTUDIO_100 -> Logos:LOGO_100
- U$15: device Logos:LOGO_100 -> Logos:WWW.DIOSTUDIO.CN_100
- U$16: device Logos:WWW.DIOSTUDIO.CN_100 -> Logos:DIOSTUDIO_100
- moved U$16 12.8 mm to (33.0, 44.5)
- moved G1 11.2 mm to (30.5, 20.3), turned to 0 degrees
- moved U$14 10.3 mm to (22.2, 44.1)
- moved U$17 7.30 mm to (44.8, 37.1)
- moved U$13 1.71 mm to (22.2, 38.4)
- moved U$15 1.42 mm to (22.2, 40.6)
- moved R10 0.64 mm to (18.4, 41.0)
- moved R11 0.64 mm to (18.4, 36.5)
- moved R12 0.64 mm to (18.4, 45.4)
- moved D1 0.64 mm to (21.0, 4.45)
- moved R1 0.64 mm to (14.3, 4.45)
- moved S1 0.64 mm to (6.35, 4.45)
- moved FUSE 0.63 mm to (21.0, 7.94)
- moved R13 0.63 mm to (18.4, 43.2)
- moved R14 0.63 mm to (18.4, 38.7)
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Connections:
- net 5V0: no longer SV2.2, SV3.2, SV4.2
- net A3: no longer SV2.3
- net D8: no longer SV3.3
- net D9: no longer SV4.3
- net GND: no longer SV2.1, SV3.1, SV4.1
Routing:
- net A3: track 65.2 -> 0.00 mm, vias 3 -> 0
- net 5V0: track 157.3 -> 125.3 mm
- net D8: track 30.1 -> 0.00 mm
- net D9: track 29.4 -> 0.00 mm
- net N$6: track 24.1 -> 36.4 mm
- net IN1: track 64.9 -> 72.0 mm
- net PWM1: track 61.1 -> 67.7 mm, vias 1 -> 0
- net 3V3: track 150.7 -> 144.7 mm, vias 2 -> 3
- net IN2: track 51.7 -> 57.0 mm, vias 0 -> 1
- net IN4: track 63.5 -> 68.6 mm
- net SS: track 23.6 -> 28.0 mm
- net OUT2: track 28.7 -> 32.8 mm
- net N$9: track 12.4 -> 8.57 mm
- net VCC: track 28.1 -> 24.4 mm, vias 0 -> 1
- net VIN: track 26.9 -> 30.2 mm
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
Commit message: 2020.07.01.02
Parts:
- added R15, R16, R17: 472, RCLDA:R0805
- turned U$23 to 90 degrees
- turned U$24 to 270 degrees
- turned U$25 to 270 degrees
Connections:
- net 5V0: now also R15.2, R16.2, R17.2
- net A3: now also R17.1, U$25.1
- net D8: now also R16.1, U$24.1
- net D9: now also R15.1, U$23.1
- net GND: now also U$23.2, U$24.2, U$25.2
Changed lines of the file:
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@@
 <element name="R13" library="RCLDA" package="R0805" value="222" x="18.415" y="43.18"/>
 <element name="R14" library="RCLDA" package="R0805" value="222" x="18.415" y="38.735"/>
-<element name="U$23" library="Button" package="TS-SMD_3*6" value="" x="40.64" y="8.89" rot="R270"/>
-<element name="U$24" library="Button" package="TS-SMD_3*6" value="" x="35.56" y="8.89" rot="R90"/>
-<element name="U$25" library="Button" package="TS-SMD_3*6" value="" x="30.48" y="8.89" rot="R90"/>
+<element name="U$23" library="Button" package="TS-SMD_3*6" value="" x="40.64" y="8.89" rot="R90"/>
+<element name="U$24" library="Button" package="TS-SMD_3*6" value="" x="35.56" y="8.89" rot="R270"/>
+<element name="U$25" library="Button" package="TS-SMD_3*6" value="" x="30.48" y="8.89" rot="R270"/>
 <element name="U$13" library="Logos" package="ARDUINO_ADVANCED_SENSOR_BOARD" value="" x="22.225" y="38.4175"/>
 <element name="U$15" library="Logos" package="WWW.DIOSTUDIO.CN_100" value="" x="22.225" y="40.64"/>
@@
 <element name="U$16" library="Logos" package="DIOSTUDIO_100" value="" x="33.02" y="44.45"/>
 <element name="U$17" library="Logos" package="MAKE_SOMETHING_FUN_100" value="" x="44.7675" y="37.1475" rot="MR0"/>
+<element name="R15" library="RCLDA" package="R0805" value="472" x="-0.3175" y="-3.4925"/>
+<element name="R16" library="RCLDA" package="R0805" value="472" x="-0.3175" y="-8.255"/>
+<element name="R17" library="RCLDA" package="R0805" value="472" x="-0.3175" y="-13.0175"/>
 </elements>
 <signals>
@@
 <wire x1="54.61" y1="44.7675" x2="53.975" y2="44.1325" width="0.6096" layer="1"/>
 <wire x1="53.975" y1="44.1325" x2="53.975" y2="42.545" width="0.6096" layer="1"/>
+<contactref element="R15" pad="2"/>
+<contactref element="R16" pad="2"/>
+<contactref element="R17" pad="2"/>
+<wire x1="0.6325" y1="-3.4925" x2="15.2375" y2="2.86" width="0" layer="19" extent="1-1"/>
+<wire x1="0.6325" y1="-8.255" x2="0.6325" y2="-3.4925" width="0" layer="19" extent="1-1"/>
+<wire x1="0.6325" y1="-13.0175" x2="0.6325" y2="-8.255" width="0" layer="19" extent="1-1"/>
 </signal>
 <signal name="GND">
@@
 <via x="6.35" y="4.445" extent="1-16" drill="0.5" shape="octagon"/>
 <via x="21.2725" y="38.735" extent="1-16" drill="0.5" shape="octagon"/>
+<contactref element="U$23" pad="2"/>
+<contactref element="U$24" pad="2"/>
+<contactref element="U$25" pad="2"/>
 </signal>
 <signal name="A3">
 <contactref element="U$1" pad="A3"/>
+<contactref element="U$25" pad="1"/>
+<contactref element="R17" pad="1"/>
+<wire x1="30.48" y1="12.7" x2="58.42" y2="2.54" width="0" layer="19" extent="1-1"/>
+<wire x1="-1.2675" y1="-13.0175" x2="30.48" y2="12.7" width="0" layer="19" extent="1-1"/>
 </signal>
 <signal name="SDA">
@@
 <signal name="D9">
 <contactref element="U$1" pad="D9"/>
+<contactref element="U$23" pad="1"/>
+<contactref element="R15" pad="1"/>
+<wire x1="40.64" y1="5.08" x2="39.37" y2="50.8" width="0" layer="19" extent="1-1"/>
+<wire x1="-1.2675" y1="-3.4925" x2="40.64" y2="5.08" width="0" layer="19" extent="1-1"/>
 </signal>
 <signal name="D8">
 <contactref element="U$1" pad="D8"/>
+<contactref element="U$24" pad="1"/>
+<contactref element="R16" pad="1"/>
+<wire x1="35.56" y1="12.7" x2="41.91" y2="50.8" width="0" layer="19" extent="1-1"/>
+<wire x1="-1.2675" y1="-8.255" x2="35.56" y2="12.7" width="0" layer="19" extent="1-1"/>
 </signal>
 </signals>

Commit message: 2020.07.02.01
Parts:
- removed D1: DIODESMB, RCLDA:SMB
- removed FUSE: F0805-1.1A, RCLDA:F0805
- removed U$23: (no value), Button:TS-SMD_3*6
- removed X1: (no value), Connector:AK500/5
- added IC1: DS18B20, Senser:TO92
- added R18: 103, RCLDA:R0805
- added SJ1, SJ2: (no value), Jumper:SJ_2
- added SV2: (no value), Pin-Header:MA04-1
- added SV3, SV4: (no value), Pin-Header:MA03-1
- added U$18: (no value), Logos:LOGO_100
- added U$19: (no value), Logos:DIOSTUDIO_100
- added U$20: (no value), Logos:WWW.DIOSTUDIO.CN_100
- added U$21, U$26: (no value), Logos:5V0_050
- added U$22: (no value), Logos:GND_050
- added U$27: (no value), Logos:D5_050
- added U$28: (no value), Logos:D4_050
- U$13: value (none) -> TS-SMD; device Logos:ARDUINO_ADVANCED_SENSOR_BOARD -> Button:TS-SMD
- U$14: value (none) -> TS-SMD; device Logos:LOGO_100 -> Button:TS-SMD
- U$15: value (none) -> IR-RECIEVER; device Logos:WWW.DIOSTUDIO.CN_100 -> Senser:IR-RECIEVER
- U$16: device Logos:DIOSTUDIO_100 -> Logos:ARDUINO_ADVANCED_SENSOR_BOARD
- U$24: device Button:TS-SMD_3*6 -> Logos:A3_050
- U$25: device Button:TS-SMD_3*6 -> Logos:GND_050
- U$3: value L293D -> TS-SMD; device Chip:DIP16 -> Button:TS-SMD
- moved R1 44.5 mm to (13.7, 48.9), turned to 90 degrees
- moved S1 44.5 mm to (6.67, 48.9)
- moved U$14 42.2 mm to (21.0, 1.91), turned to 180 degrees
- moved U$16 41.2 mm to (10.2, 10.2)
- moved U$13 37.7 mm to (12.7, 1.91), turned to 180 degrees
- moved R17 29.0 mm to (21.0, 6.67), flipped to the bottom, turned to 90 degrees
- moved U$25 27.0 mm to (5.71, 19.7), turned to 0 degrees
- moved U$17 23.3 mm to (42.5, 14.0)
- moved U$3 21.9 mm to (4.45, 1.91), turned to 180 degrees
- moved R16 19.8 mm to (12.7, 6.67), flipped to the bottom, turned to 90 degrees
- moved U$15 18.2 mm to (30.5, 24.4)
- moved G1 11.4 mm to (30.5, 31.8)
- moved R15 11.2 mm to (4.45, 6.67), flipped to the bottom, turned to 90 degrees
- moved U$24 7.68 mm to (42.2, 12.7), turned to 0 degrees
- moved R10 7.62 mm to (18.4, 33.3)
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Connections:
- removed net IN1: U$1.D2, U$3.2
- removed net IN2: U$1.D3, U$3.7
- removed net IN3: U$1.D4, U$3.10
- removed net IN4: U$1.D7, U$3.15
- removed net N$1: D1.1, FUSE.1
- removed net N$2: U$1.REF
- removed net N$3: U$1.AREF
- removed net OUT1: U$3.3, X1.1
- removed net OUT2: U$3.6, X1.2
- removed net OUT3: U$3.11, X1.4
- removed net OUT4: U$3.14, X1.5
- removed net PWM1: U$1.D5, U$3.1
- removed net PWM2: U$1.D6, U$3.9
- removed net VCC: FUSE.2, U$3.8
- new net AREF: SJ2.2, U$1.AREF
- new net D2: IC1.2, R18.1, U$1.D2
- new net D3: U$1.D3, U$15.OUT
- new net D4: SV3.3, U$1.D4
- new net D5: R17.1, U$1.D5, U$14.P
- new net D6: R16.1, U$1.D6, U$13.P
- new net D7: R15.1, U$1.D7, U$3.P
- new net DREF: SJ1.2, U$1.REF
- net 3V3: now also SJ1.1, SJ2.1
- net 5V0: now also IC1.3, R18.2, SJ1.3, SJ2.3, SV2.4, SV3.2, SV4.2, U$15.VCC; no longer U$3.16
- net A3: now also SV4.3; no longer R17.1, U$25.1
- net D8: now also SV2.3; no longer R16.1, U$24.1
- net D9: now also SV2.2; no longer R15.1, U$23.1
- net GND: now also IC1.1, SV2.1, SV3.1, SV4.1, U$13.S, U$14.S, U$15.GND, U$3.S; no longer U$23.2, U$24.2, U$25.2, U$3.12, U$3.13, U$3.4, U$3.5, X1.3
- net VIN: no longer D1.2
Routing:
- net D7: track 0.00 -> 84.9 mm, vias 0 -> 1
- net D6: track 0.00 -> 80.9 mm, vias 0 -> 1
- net D5: track 0.00 -> 75.9 mm, vias 0 -> 1
- net IN1: track 72.0 -> 0.00 mm, vias 1 -> 0
- net D8: track 0.00 -> 69.2 mm
- net IN4: track 68.6 -> 0.00 mm, vias 1 -> 0
- net PWM1: track 67.7 -> 0.00 mm
- net D9: track 0.00 -> 65.2 mm
- net D4: track 0.00 -> 62.2 mm, vias 0 -> 1
- net IN3: track 61.9 -> 0.00 mm, vias 1 -> 0
- net IN2: track 57.0 -> 0.00 mm, vias 1 -> 0
- net D3: track 0.00 -> 54.9 mm, vias 0 -> 1
- net PWM2: track 53.7 -> 0.00 mm
- net 3V3: track 144.7 -> 94.4 mm, vias 3 -> 2
- net RESET: track 38.0 -> 81.1 mm, vias 1 -> 2
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
Commit message: 2020.07.03.02
Parts:
- added U$23: (no value), Logos:D4_050
- moved U$17 1.91 mm to (42.5, 12.1)
- moved U$16 0.63 mm to (9.53, 10.2)
- moved U$18 0.63 mm to (9.53, 16.5)
- moved U$20 0.63 mm to (9.53, 12.7)
- moved U$19 0.63 mm to (20.3, 16.8)
Routing:
- net 3V3: track 94.4 -> 188.7 mm, vias 2 -> 4
- net A3: track 0.00 -> 47.2 mm
- net 5V0: track 142.6 -> 183.9 mm, vias 2 -> 4
- net SDA: track 7.80 -> 41.6 mm, vias 0 -> 1
- net SCL: track 6.76 -> 38.5 mm
- net D2: track 27.0 -> 25.4 mm
- net MISO: track 26.9 -> 26.2 mm
