File: projects/03 Arduino Advanced Sensor Board/Arduino Advanced Sensor Board.sch (EAGLE design)
At the start: 28 parts

Commit message: 2020.06.16.01
Parts:
- added R10, R11, R9: 102, RCLDA:R0805
- added R12, R13, R14: 222, RCLDA:R0805
Connections:
- removed net A0: U$1.A0
- removed net A1: U$1.A1
- removed net A2: U$1.A2
- removed net D2: U$1.D2
- removed net D3: U$1.D3/PWM
- removed net D4: U$1.D4
- new net MISO: SD1.DO, U$1.D12/MISO
- new net MOSI: R10.1, U$1.D11/PWM/MOSI
- new net N$10: R10.2, R13.1, SD1.DI
- new net N$12: R12.1, R9.2, SD1.SCLK
- new net N$9: R11.2, R14.1, SD1.CS
- new net SCK: R9.1, U$1.D13/SCK
- new net SS: R11.1, U$1.D10/PWM/SS
- net 3V3: now also SD1.VDD
- net CE: now also U$1.A0; no longer U$1.D5/PWM
- net GND: now also R12.2, R13.2, R14.2, SD1.G1, SD1.G2, SD1.G3, SD1.G4, SD1.VSS
- net IN1: now also U$1.D2; no longer U$1.D13/SCK
- net IN2: now also U$1.D3/PWM; no longer U$1.D12/MISO
- net IN3: now also U$1.D4; no longer U$1.D9/PWM
- net IN4: now also U$1.D7; no longer U$1.D8
- net IO: now also U$1.A1; no longer U$1.D6/PWM
- net PWM1: now also U$1.D5/PWM; no longer U$1.D11/PWM/MOSI
- net PWM2: now also U$1.D6/PWM; no longer U$1.D10/PWM/SS
- net SCLK: now also U$1.A2; no longer U$1.D7
Other:
- note added: "microSD"
- moved on the sheet: SD1

Commit message: 2020.06.26.01
Parts:
- added SV3, SV4: (no value), Pin-Header:MA03-1
Connections:
- new net D8: SV3.3, U$1.D8
- new net D9: SV4.3, U$1.D9/PWM
- net 5V0: now also SV3.2, SV4.2
- net GND: now also SV3.1, SV4.1
Changed lines of the file:
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@@
 <part name="R13" library="RCLDA" deviceset="R" device="0805" value="222"/>
 <part name="R14" library="RCLDA" deviceset="R" device="0805" value="222"/>
+<part name="SV3" library="Pin-Header" deviceset="MA03-1" device=""/>
+<part name="SV4" library="Pin-Header" deviceset="MA03-1" device=""/>
 </parts>
 <sheets>
@@
 <instance part="R13" gate="G$1" x="102.87" y="165.1" rot="R180"/>
 <instance part="R14" gate="G$1" x="102.87" y="158.75" rot="R180"/>
+<instance part="SV3" gate="G$1" x="46.99" y="95.25"/>
+<instance part="SV4" gate="G$1" x="64.77" y="95.25"/>
 </instances>
 <busses>
@@
 <wire x1="215.9" y1="49.53" x2="222.25" y2="49.53" width="0.1524" layer="91"/>
 <label x="215.9" y="49.53" size="1.27" layer="95"/>
+</segment>
+<segment>
+<pinref part="SV4" gate="G$1" pin="2"/>
+<wire x1="78.74" y1="95.25" x2="72.39" y2="95.25" width="0.1524" layer="91"/>
+<label x="73.66" y="95.25" size="1.27" layer="95"/>
+</segment>
+<segment>
+<pinref part="SV3" gate="G$1" pin="2"/>
+<wire x1="60.96" y1="95.25" x2="54.61" y2="95.25" width="0.1524" layer="91"/>
+<label x="55.88" y="95.25" size="1.27" layer="95"/>
 </segment>
 </net>
@@
 <junction x="153.67" y="152.4"/>
 <label x="143.51" y="152.4" size="1.27" layer="95"/>
+</segment>
+<segment>
+<pinref part="SV3" gate="G$1" pin="1"/>
+<wire x1="60.96" y1="92.71" x2="54.61" y2="92.71" width="0.1524" layer="91"/>
+<label x="55.88" y="92.71" size="1.27" layer="95"/>
+</segment>
+<segment>
+<pinref part="SV4" gate="G$1" pin="1"/>
+<wire x1="78.74" y1="92.71" x2="72.39" y2="92.71" width="0.1524" layer="91"/>
+<label x="73.66" y="92.71" size="1.27" layer="95"/>
 </segment>
 </net>
@@
 </segment>
 </net>
+<net name="D9" class="0">
+<segment>
+<pinref part="U$1" gate="G$1" pin="D9/PWM"/>
+<wire x1="67.31" y1="135.89" x2="60.96" y2="135.89" width="0.1524" layer="91"/>
+<label x="62.23" y="135.89" size="1.27" layer="95"/>
+</segment>
+<segment>
+<pinref part="SV4" gate="G$1" pin="3"/>
+<wire x1="78.74" y1="97.79" x2="72.39" y2="97.79" width="0.1524" layer="91"/>
+<label x="73.66" y="97.79" size="1.27" layer="95"/>
+</segment>
+</net>
+<net name="D8" class="0">
+<segment>
+<pinref part="U$1" gate="G$1" pin="D8"/>
+<wire x1="67.31" y1="133.35" x2="60.96" y2="133.35" width="0.1524" layer="91"/>
+<label x="62.23" y="133.35" size="1.27" layer="95"/>
+</segment>
+<segment>
+<pinref part="SV3" gate="G$1" pin="3"/>
+<wire x1="60.96" y1="97.79" x2="54.61" y2="97.79" width="0.1524" layer="91"/>
+<label x="55.88" y="97.79" size="1.27" layer="95"/>
+</segment>
+</net>

Commit message: 2020.06.30.01
Parts:
- added SV2: (no value), Pin-Header:MA03-1
Connections:
- net 5V0: now also SV2.2
- net A3: now also SV2.3
- net GND: now also SV2.1
Changed lines of the file:
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@@
 <part name="SV3" library="Pin-Header" deviceset="MA03-1" device=""/>
 <part name="SV4" library="Pin-Header" deviceset="MA03-1" device=""/>
+<part name="SV2" library="Pin-Header" deviceset="MA03-1" device=""/>
 </parts>
 <sheets>
@@
 <instance part="SV3" gate="G$1" x="46.99" y="95.25"/>
 <instance part="SV4" gate="G$1" x="64.77" y="95.25"/>
+<instance part="SV2" gate="G$1" x="87.63" y="95.25"/>
 </instances>
 <busses>
@@
 <wire x1="60.96" y1="95.25" x2="54.61" y2="95.25" width="0.1524" layer="91"/>
 <label x="55.88" y="95.25" size="1.27" layer="95"/>
+</segment>
+<segment>
+<pinref part="SV2" gate="G$1" pin="2"/>
+<wire x1="101.6" y1="95.25" x2="95.25" y2="95.25" width="0.1524" layer="91"/>
+<label x="96.52" y="95.25" size="1.27" layer="95"/>
 </segment>
 </net>
@@
 <label x="73.66" y="92.71" size="1.27" layer="95"/>
 </segment>
+<segment>
+<pinref part="SV2" gate="G$1" pin="1"/>
+<wire x1="101.6" y1="92.71" x2="95.25" y2="92.71" width="0.1524" layer="91"/>
+<label x="96.52" y="92.71" size="1.27" layer="95"/>
+</segment>
 </net>
 <net name="A3" class="0">
@@
 <label x="20.32" y="118.11" size="1.27" layer="95"/>
 </segment>
-</net>
+<segment>
+<pinref part="SV2" gate="G$1" pin="3"/>
+<wire x1="101.6" y1="97.79" x2="95.25" y2="97.79" width="0.1524" layer="91"/>
+<label x="96.52" y="97.79" size="1.27" layer="95"/>
+</segment>
+</net>

Commit message: 2020.07.01.01
Parts:
- removed SV2, SV3, SV4: (no value), Pin-Header:MA03-1
- added U$23, U$24, U$25: TS-SMD_36TS-SMD-3*6, Button:TS-SMD_36TS-SMD-3*6
Connections:
- net 5V0: no longer SV2.2, SV3.2, SV4.2
- net A3: no longer SV2.3
- net D8: no longer SV3.3
- net D9: no longer SV4.3
- net GND: no longer SV2.1, SV3.1, SV4.1
Changed lines of the file:
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@@
 <setting verticaltext="up"/>
 </settings>
-<grid distance="50" unitdist="mil" unit="mil" style="lines" multiple="1" display="yes" altdistance="25" altunitdist="mil" altunit="mil"/>
+<grid distance="0.1" unitdist="inch" unit="inch" style="lines" multiple="1" display="no" altdistance="0.01" altunitdist="inch" altunit="inch"/>
 <layers>
 <layer number="1" name="Top" color="4" fill="1" visible="no" active="no"/>
@@
 <part name="R13" library="RCLDA" deviceset="R" device="0805" value="222"/>
 <part name="R14" library="RCLDA" deviceset="R" device="0805" value="222"/>
-<part name="SV3" library="Pin-Header" deviceset="MA03-1" device=""/>
-<part name="SV4" library="Pin-Header" deviceset="MA03-1" device=""/>
-<part name="SV2" library="Pin-Header" deviceset="MA03-1" device=""/>
+<part name="U$23" library="Button" deviceset="TS-SMD_3*6" device="TS-SMD-3*6" value=""/>
+<part name="U$24" library="Button" deviceset="TS-SMD_3*6" device="TS-SMD-3*6" value=""/>
+<part name="U$25" library="Button" deviceset="TS-SMD_3*6" device="TS-SMD-3*6" value=""/>
 </parts>
 <sheets>
@@
 <instance part="R13" gate="G$1" x="102.87" y="165.1" rot="R180"/>
 <instance part="R14" gate="G$1" x="102.87" y="158.75" rot="R180"/>
-<instance part="SV3" gate="G$1" x="46.99" y="95.25"/>
-<instance part="SV4" gate="G$1" x="64.77" y="95.25"/>
-<instance part="SV2" gate="G$1" x="87.63" y="95.25"/>
+<instance part="U$23" gate="G$1" x="35.56" y="76.2"/>
+<instance part="U$24" gate="G$1" x="53.34" y="76.2"/>
+<instance part="U$25" gate="G$1" x="81.28" y="78.74"/>
 </instances>
 <busses>
@@
 <wire x1="215.9" y1="49.53" x2="222.25" y2="49.53" width="0.1524" layer="91"/>
 <label x="215.9" y="49.53" size="1.27" layer="95"/>
-</segment>
-<segment>
-<pinref part="SV4" gate="G$1" pin="2"/>
-<wire x1="78.74" y1="95.25" x2="72.39" y2="95.25" width="0.1524" layer="91"/>
-<label x="73.66" y="95.25" size="1.27" layer="95"/>
-</segment>
-<segment>
-<pinref part="SV3" gate="G$1" pin="2"/>
-<wire x1="60.96" y1="95.25" x2="54.61" y2="95.25" width="0.1524" layer="91"/>
-<label x="55.88" y="95.25" size="1.27" layer="95"/>
-</segment>
-<segment>
-<pinref part="SV2" gate="G$1" pin="2"/>
-<wire x1="101.6" y1="95.25" x2="95.25" y2="95.25" width="0.1524" layer="91"/>
-<label x="96.52" y="95.25" size="1.27" layer="95"/>
 </segment>
 </net>
@@
 <label x="143.51" y="152.4" size="1.27" layer="95"/>
 </segment>
-<segment>
-<pinref part="SV3" gate="G$1" pin="1"/>
-<wire x1="60.96" y1="92.71" x2="54.61" y2="92.71" width="0.1524" layer="91"/>
-<label x="55.88" y="92.71" size="1.27" layer="95"/>
-</segment>
-<segment>
-<pinref part="SV4" gate="G$1" pin="1"/>
-<wire x1="78.74" y1="92.71" x2="72.39" y2="92.71" width="0.1524" layer="91"/>
-<label x="73.66" y="92.71" size="1.27" layer="95"/>
-</segment>
-<segment>
-<pinref part="SV2" gate="G$1" pin="1"/>
-<wire x1="101.6" y1="92.71" x2="95.25" y2="92.71" width="0.1524" layer="91"/>
-<label x="96.52" y="92.71" size="1.27" layer="95"/>
-</segment>
 </net>
 <net name="A3" class="0">
@@
 <wire x1="25.4" y1="118.11" x2="20.32" y2="118.11" width="0.1524" layer="91"/>
 <label x="20.32" y="118.11" size="1.27" layer="95"/>
-</segment>
-<segment>
-<pinref part="SV2" gate="G$1" pin="3"/>
-<wire x1="101.6" y1="97.79" x2="95.25" y2="97.79" width="0.1524" layer="91"/>
-<label x="96.52" y="97.79" size="1.27" layer="95"/>
 </segment>
 </net>
@@
 <label x="62.23" y="135.89" size="1.27" layer="95"/>
 </segment>
-<segment>
-<pinref part="SV4" gate="G$1" pin="3"/>
-<wire x1="78.74" y1="97.79" x2="72.39" y2="97.79" width="0.1524" layer="91"/>
-<label x="73.66" y="97.79" size="1.27" layer="95"/>
-</segment>
 </net>
 <net name="D8" class="0">
@@
 <label x="62.23" y="133.35" size="1.27" layer="95"/>
 </segment>
-<segment>
-<pinref part="SV3" gate="G$1" pin="3"/>
-<wire x1="60.96" y1="97.79" x2="54.61" y2="97.79" width="0.1524" layer="91"/>
-<label x="55.88" y="97.79" size="1.27" layer="95"/>
-</segment>
-</net>
+</net>

Commit message: 2020.07.01.02
Parts:
- added R15, R16, R17: 472, RCLDA:R0805
Connections:
- net 5V0: now also R15.2, R16.2, R17.2
- net A3: now also R17.1, U$25.P
- net D8: now also R16.1, U$24.P
- net D9: now also R15.1, U$23.P
- net GND: now also U$23.S, U$24.S, U$25.S
Other:
- moved on the sheet: U$23, U$24, U$25
Changed lines of the file:
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@@
 <setting verticaltext="up"/>
 </settings>
-<grid distance="0.1" unitdist="inch" unit="inch" style="lines" multiple="1" display="no" altdistance="0.01" altunitdist="inch" altunit="inch"/>
+<grid distance="50" unitdist="mil" unit="mil" style="lines" multiple="1" display="yes" altdistance="0.01" altunitdist="inch" altunit="mil"/>
 <layers>
 <layer number="1" name="Top" color="4" fill="1" visible="no" active="no"/>
@@
 <part name="U$24" library="Button" deviceset="TS-SMD_3*6" device="TS-SMD-3*6" value=""/>
 <part name="U$25" library="Button" deviceset="TS-SMD_3*6" device="TS-SMD-3*6" value=""/>
+<part name="R15" library="RCLDA" deviceset="R" device="0805" value="472"/>
+<part name="R16" library="RCLDA" deviceset="R" device="0805" value="472"/>
+<part name="R17" library="RCLDA" deviceset="R" device="0805" value="472"/>
 </parts>
 <sheets>
@@
 <instance part="R13" gate="G$1" x="102.87" y="165.1" rot="R180"/>
 <instance part="R14" gate="G$1" x="102.87" y="158.75" rot="R180"/>
-<instance part="U$23" gate="G$1" x="35.56" y="76.2"/>
-<instance part="U$24" gate="G$1" x="53.34" y="76.2"/>
-<instance part="U$25" gate="G$1" x="81.28" y="78.74"/>
+<instance part="U$23" gate="G$1" x="43.18" y="96.52"/>
+<instance part="U$24" gate="G$1" x="43.18" y="85.09"/>
+<instance part="U$25" gate="G$1" x="43.18" y="73.66"/>
+<instance part="R15" gate="G$1" x="26.67" y="96.52" rot="R180"/>
+<instance part="R16" gate="G$1" x="26.67" y="85.09" rot="R180"/>
+<instance part="R17" gate="G$1" x="26.67" y="73.66" rot="R180"/>
 </instances>
 <busses>
@@
 <wire x1="215.9" y1="49.53" x2="222.25" y2="49.53" width="0.1524" layer="91"/>
 <label x="215.9" y="49.53" size="1.27" layer="95"/>
+</segment>
+<segment>
+<pinref part="R15" gate="G$1" pin="2"/>
+<wire x1="16.51" y1="96.52" x2="21.59" y2="96.52" width="0.1524" layer="91"/>
+<label x="16.51" y="96.52" size="1.27" layer="95"/>
+</segment>
+<segment>
+<pinref part="R16" gate="G$1" pin="2"/>
+<wire x1="16.51" y1="85.09" x2="21.59" y2="85.09" width="0.1524" layer="91"/>
+<label x="16.51" y="85.09" size="1.27" layer="95"/>
+</segment>
+<segment>
+<pinref part="R17" gate="G$1" pin="2"/>
+<wire x1="16.51" y1="73.66" x2="21.59" y2="73.66" width="0.1524" layer="91"/>
+<label x="16.51" y="73.66" size="1.27" layer="95"/>
 </segment>
 </net>
@@
 <label x="143.51" y="152.4" size="1.27" layer="95"/>
 </segment>
+<segment>
+<pinref part="U$23" gate="G$1" pin="S"/>
+<wire x1="53.34" y1="96.52" x2="48.26" y2="96.52" width="0.1524" layer="91"/>
+<label x="49.53" y="96.52" size="1.27" layer="95"/>
+</segment>
+<segment>
+<pinref part="U$24" gate="G$1" pin="S"/>
+<wire x1="53.34" y1="85.09" x2="48.26" y2="85.09" width="0.1524" layer="91"/>
+<label x="49.53" y="85.09" size="1.27" layer="95"/>
+</segment>
+<segment>
+<pinref part="U$25" gate="G$1" pin="S"/>
+<wire x1="53.34" y1="73.66" x2="48.26" y2="73.66" width="0.1524" layer="91"/>
+<label x="49.53" y="73.66" size="1.27" layer="95"/>
+</segment>
 </net>
 <net name="A3" class="0">
@@
 <wire x1="25.4" y1="118.11" x2="20.32" y2="118.11" width="0.1524" layer="91"/>
 <label x="20.32" y="118.11" size="1.27" layer="95"/>
+</segment>
+<segment>
+<pinref part="U$25" gate="G$1" pin="P"/>
+<wire x1="31.75" y1="73.66" x2="38.1" y2="73.66" width="0.1524" layer="91"/>
+<pinref part="R17" gate="G$1" pin="1"/>
+<label x="33.02" y="73.66" size="1.27" layer="95"/>
 </segment>
 </net>
@@
 <label x="62.23" y="135.89" size="1.27" layer="95"/>
 </segment>
+<segment>
+<pinref part="U$23" gate="G$1" pin="P"/>
+<pinref part="R15" gate="G$1" pin="1"/>
+<wire x1="31.75" y1="96.52" x2="38.1" y2="96.52" width="0.1524" layer="91"/>
+<label x="33.02" y="96.52" size="1.27" layer="95"/>
+</segment>
 </net>
 <net name="D8" class="0">
@@
 <label x="62.23" y="133.35" size="1.27" layer="95"/>
 </segment>
-</net>
+<segment>
+<pinref part="U$24" gate="G$1" pin="P"/>
+<wire x1="31.75" y1="85.09" x2="38.1" y2="85.09" width="0.1524" layer="91"/>
+<pinref part="R16" gate="G$1" pin="1"/>
+<label x="33.02" y="85.09" size="1.27" layer="95"/>
+</segment>
+</net>

Commit message: 2020.07.02.01
Parts:
- removed D1: DIODESMB, RCLDA:DIODESMB
- removed FUSE: F0805-1.1A, RCLDA:FUSE0805
- removed U$23, U$24, U$25: TS-SMD_36TS-SMD-3*6, Button:TS-SMD_36TS-SMD-3*6
- removed X1: (no value), Connector:AK500/5
- added IC1: DS18B20, Senser:DS18B20
- added R18: 103, RCLDA:R0805
- added SJ1, SJ2: (no value), Jumper:SJ2W
- added SV2: (no value), Pin-Header:MA04-1
- added SV3, SV4: (no value), Pin-Header:MA03-1
- added U$13, U$14: TS-SMD, Button:TS-SMD
- added U$15: IR-RECIEVER, Senser:IR-RECIEVER
- U$3: value L293D -> TS-SMD; device Chip:L293D -> Button:TS-SMD
Connections:
- removed net IN1: U$1.D2, U$3.IN1
- removed net IN2: U$1.D3/PWM, U$3.IN2
- removed net IN3: U$1.D4, U$3.IN3
- removed net IN4: U$1.D7, U$3.IN4
- removed net N$1: D1.1, FUSE.P$1
- removed net N$2: U$1.IOREF
- removed net N$3: U$1.AREF
- removed net OUT1: U$3.OUT1, X1-1.KL
- removed net OUT2: U$3.OUT2, X1-2.KL
- removed net OUT3: U$3.OUT3, X1-4.KL
- removed net OUT4: U$3.OUT4, X1-5.KL
- removed net PWM1: U$1.D5/PWM, U$3.EN1
- removed net PWM2: U$1.D6/PWM, U$3.EN2
- removed net VCC: FUSE.P$2, U$3.VS
- new net AREF: SJ2.2, U$1.AREF
- new net D2: IC1.DQ, R18.1, U$1.D2
- new net D3: U$1.D3/PWM, U$15.OUT
- new net D4: SV3.3, U$1.D4
- new net D5: R17.1, U$1.D5/PWM, U$14.P
- new net D6: R16.1, U$1.D6/PWM, U$13.P
- new net D7: R15.1, U$1.D7, U$3.P
- new net DREF: SJ1.2, U$1.IOREF
- net 3V3: now also SJ1.1, SJ2.1
- net 5V0: now also IC1.VCC, R18.2, SJ1.3, SJ2.3, SV2.4, SV3.2, SV4.2, U$15.VCC; no longer U$3.VSS
- net A3: now also SV4.3; no longer R17.1, U$25.P
- net D8: now also SV2.3; no longer R16.1, U$24.P
- net D9: now also SV2.2; no longer R15.1, U$23.P
- net GND: now also IC1.GND, SV2.1, SV3.1, SV4.1, U$13.S, U$14.S, U$15.GND, U$3.S; no longer U$23.S, U$24.S, U$25.S, U$3.GND@1, U$3.GND@2, U$3.GND@3, U$3.GND@4, X1-3.KL
- net VIN: no longer D1.2
Other:
- note removed: "L293D"
- moved on the sheet: R15, R16, R17, U$1
