File: projects/02 Arduino Basic Sensor Board/Arduino Basic Sensor Board.brd (EAGLE design)
At the start: 68.6 x 53.3 mm, 85 parts, among them Q1 S8050SOT23, Q2 S8050SOT23

Commit message: 2020.06.12.01
Parts:
- U$8: device Chip:SO16 -> Chip:SOP16
Changed lines of the file:
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@@
 <layer number="15" name="Route15" color="4" fill="6" visible="no" active="no"/>
 <layer number="16" name="Bottom" color="1" fill="1" visible="yes" active="yes"/>
-<layer number="17" name="Pads" color="2" fill="1" visible="yes" active="yes"/>
-<layer number="18" name="Vias" color="2" fill="1" visible="yes" active="yes"/>
+<layer number="17" name="Pads" color="2" fill="1" visible="no" active="yes"/>
+<layer number="18" name="Vias" color="2" fill="1" visible="no" active="yes"/>
 <layer number="19" name="Unrouted" color="6" fill="1" visible="yes" active="yes"/>
 <layer number="20" name="Dimension" color="15" fill="1" visible="yes" active="yes"/>
 <layer number="21" name="tPlace" color="7" fill="1" visible="yes" active="yes"/>
 <layer number="22" name="bPlace" color="7" fill="1" visible="yes" active="yes"/>
-<layer number="23" name="tOrigins" color="15" fill="1" visible="yes" active="yes"/>
-<layer number="24" name="bOrigins" color="15" fill="1" visible="yes" active="yes"/>
+<layer number="23" name="tOrigins" color="15" fill="1" visible="no" active="yes"/>
+<layer number="24" name="bOrigins" color="15" fill="1" visible="no" active="yes"/>
 <layer number="25" name="tNames" color="7" fill="1" visible="no" active="yes"/>
 <layer number="26" name="bNames" color="7" fill="1" visible="no" active="yes"/>
 <layer number="27" name="tValues" color="7" fill="1" visible="no" active="yes"/>
 <layer number="28" name="bValues" color="7" fill="1" visible="no" active="yes"/>
-<layer number="29" name="tStop" color="7" fill="3" visible="yes" active="yes"/>
-<layer number="30" name="bStop" color="7" fill="6" visible="yes" active="yes"/>
-<layer number="31" name="tCream" color="7" fill="4" visible="yes" active="yes"/>
-<layer number="32" name="bCream" color="7" fill="5" visible="yes" active="yes"/>
-<layer number="33" name="tFinish" color="6" fill="3" visible="yes" active="yes"/>
-<layer number="34" name="bFinish" color="6" fill="6" visible="yes" active="yes"/>
-<layer number="35" name="tGlue" color="7" fill="4" visible="yes" active="yes"/>
-<layer number="36" name="bGlue" color="7" fill="5" visible="yes" active="yes"/>
-<layer number="37" name="tTest" color="7" fill="1" visible="yes" active="yes"/>
-<layer number="38" name="bTest" color="7" fill="1" visible="yes" active="yes"/>
-<layer number="39" name="tKeepout" color="4" fill="11" visible="yes" active="yes"/>
-<layer number="40" name="bKeepout" color="1" fill="11" visible="yes" active="yes"/>
-<layer number="41" name="tRestrict" color="4" fill="10" visible="yes" active="yes"/>
-<layer number="42" name="bRestrict" color="1" fill="10" visible="yes" active="yes"/>
-<layer number="43" name="vRestrict" color="2" fill="10" visible="yes" active="yes"/>
-<layer number="44" name="Drills" color="7" fill="1" visible="yes" active="yes"/>
-<layer number="45" name="Holes" color="7" fill="1" visible="yes" active="yes"/>
-<layer number="46" name="Milling" color="3" fill="1" visible="yes" active="yes"/>
-<layer number="47" name="Measures" color="7" fill="1" visible="yes" active="yes"/>
-<layer number="48" name="Document" color="7" fill="1" visible="yes" active="yes"/>
-<layer number="49" name="Reference" color="7" fill="1" visible="yes" active="yes"/>
+<layer number="29" name="tStop" color="7" fill="3" visible="no" active="yes"/>
+<layer number="30" name="bStop" color="7" fill="6" visible="no" active="yes"/>
+<layer number="31" name="tCream" color="7" fill="4" visible="no" active="yes"/>
+<layer number="32" name="bCream" color="7" fill="5" visible="no" active="yes"/>
+<layer number="33" name="tFinish" color="6" fill="3" visible="no" active="yes"/>
+<layer number="34" name="bFinish" color="6" fill="6" visible="no" active="yes"/>
+<layer number="35" name="tGlue" color="7" fill="4" visible="no" active="yes"/>
+<layer number="36" name="bGlue" color="7" fill="5" visible="no" active="yes"/>
+<layer number="37" name="tTest" color="7" fill="1" visible="no" active="yes"/>
+<layer number="38" name="bTest" color="7" fill="1" visible="no" active="yes"/>
+<layer number="39" name="tKeepout" color="4" fill="11" visible="no" active="yes"/>
+<layer number="40" name="bKeepout" color="1" fill="11" visible="no" active="yes"/>
+<layer number="41" name="tRestrict" color="4" fill="10" visible="no" active="yes"/>
+<layer number="42" name="bRestrict" color="1" fill="10" visible="no" active="yes"/>
+<layer number="43" name="vRestrict" color="2" fill="10" visible="no" active="yes"/>
+<layer number="44" name="Drills" color="7" fill="1" visible="no" active="yes"/>
+<layer number="45" name="Holes" color="7" fill="1" visible="no" active="yes"/>
+<layer number="46" name="Milling" color="3" fill="1" visible="no" active="yes"/>
+<layer number="47" name="Measures" color="7" fill="1" visible="no" active="yes"/>
+<layer number="48" name="Document" color="7" fill="1" visible="no" active="yes"/>
+<layer number="49" name="Reference" color="7" fill="1" visible="no" active="yes"/>
 <layer number="50" name="dxf" color="7" fill="1" visible="no" active="no"/>
 <layer number="51" name="tDocu" color="7" fill="1" visible="yes" active="yes"/>
@@
 <element name="U$45" library="Logos" package="RED_050" value="" x="1.27" y="50.165"/>
 <element name="U$46" library="Logos" package="YELLOW_050" value="" x="1.27" y="47.625"/>
-<element name="U$8" library="Chip" package="SO16" value="TM1650" x="57.15" y="15.875" rot="R180"/>
+<element name="U$8" library="Chip" package="SOP16" value="TM1650" x="57.15" y="15.875" rot="R180"/>
 <element name="S3" library="Button" package="TS-SMD_6*6_SHIELD" value="TS-SMD_6S6_SHIELD" x="6.35" y="4.445"/>
 <element name="R12" library="RCLDA" package="R0805" value="103" x="13.97" y="4.445" rot="R270"/>

Commit message: 2020.06.19.01
Parts:
- D1: value DIODESMB -> (none)
- Q1, Q2: value S8050SOT23 -> (none)
- S3: value TS-SMD_6S6_SHIELD -> (none)
- U$1: value ARDUINO-UNO -> (none)
- U$15: value 3261AS -> (none)
- U$2: value 33623362 -> (none)
- U$3: value BUZZER -> (none)
- U$4: value DHT11 -> (none)
- U$5: value LM35 -> (none)
- U$6: value LDR -> (none)
- U$8: value TM1650 -> (none)
Changed lines of the file:
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@@
 <layer number="15" name="Route15" color="4" fill="6" visible="no" active="no"/>
 <layer number="16" name="Bottom" color="1" fill="1" visible="yes" active="yes"/>
-<layer number="17" name="Pads" color="2" fill="1" visible="no" active="yes"/>
-<layer number="18" name="Vias" color="2" fill="1" visible="no" active="yes"/>
+<layer number="17" name="Pads" color="2" fill="1" visible="yes" active="yes"/>
+<layer number="18" name="Vias" color="2" fill="1" visible="yes" active="yes"/>
 <layer number="19" name="Unrouted" color="6" fill="1" visible="yes" active="yes"/>
 <layer number="20" name="Dimension" color="15" fill="1" visible="yes" active="yes"/>
 <layer number="21" name="tPlace" color="7" fill="1" visible="yes" active="yes"/>
 <layer number="22" name="bPlace" color="7" fill="1" visible="yes" active="yes"/>
-<layer number="23" name="tOrigins" color="15" fill="1" visible="no" active="yes"/>
-<layer number="24" name="bOrigins" color="15" fill="1" visible="no" active="yes"/>
+<layer number="23" name="tOrigins" color="15" fill="1" visible="yes" active="yes"/>
+<layer number="24" name="bOrigins" color="15" fill="1" visible="yes" active="yes"/>
 <layer number="25" name="tNames" color="7" fill="1" visible="no" active="yes"/>
 <layer number="26" name="bNames" color="7" fill="1" visible="no" active="yes"/>
 <layer number="27" name="tValues" color="7" fill="1" visible="no" active="yes"/>
 <layer number="28" name="bValues" color="7" fill="1" visible="no" active="yes"/>
-<layer number="29" name="tStop" color="7" fill="3" visible="no" active="yes"/>
-<layer number="30" name="bStop" color="7" fill="6" visible="no" active="yes"/>
-<layer number="31" name="tCream" color="7" fill="4" visible="no" active="yes"/>
-<layer number="32" name="bCream" color="7" fill="5" visible="no" active="yes"/>
-<layer number="33" name="tFinish" color="6" fill="3" visible="no" active="yes"/>
-<layer number="34" name="bFinish" color="6" fill="6" visible="no" active="yes"/>
-<layer number="35" name="tGlue" color="7" fill="4" visible="no" active="yes"/>
-<layer number="36" name="bGlue" color="7" fill="5" visible="no" active="yes"/>
-<layer number="37" name="tTest" color="7" fill="1" visible="no" active="yes"/>
-<layer number="38" name="bTest" color="7" fill="1" visible="no" active="yes"/>
-<layer number="39" name="tKeepout" color="4" fill="11" visible="no" active="yes"/>
-<layer number="40" name="bKeepout" color="1" fill="11" visible="no" active="yes"/>
-<layer number="41" name="tRestrict" color="4" fill="10" visible="no" active="yes"/>
-<layer number="42" name="bRestrict" color="1" fill="10" visible="no" active="yes"/>
-<layer number="43" name="vRestrict" color="2" fill="10" visible="no" active="yes"/>
-<layer number="44" name="Drills" color="7" fill="1" visible="no" active="yes"/>
-<layer number="45" name="Holes" color="7" fill="1" visible="no" active="yes"/>
-<layer number="46" name="Milling" color="3" fill="1" visible="no" active="yes"/>
-<layer number="47" name="Measures" color="7" fill="1" visible="no" active="yes"/>
-<layer number="48" name="Document" color="7" fill="1" visible="no" active="yes"/>
-<layer number="49" name="Reference" color="7" fill="1" visible="no" active="yes"/>
+<layer number="29" name="tStop" color="7" fill="3" visible="yes" active="yes"/>
+<layer number="30" name="bStop" color="7" fill="6" visible="yes" active="yes"/>
+<layer number="31" name="tCream" color="7" fill="4" visible="yes" active="yes"/>
+<layer number="32" name="bCream" color="7" fill="5" visible="yes" active="yes"/>
+<layer number="33" name="tFinish" color="6" fill="3" visible="yes" active="yes"/>
+<layer number="34" name="bFinish" color="6" fill="6" visible="yes" active="yes"/>
+<layer number="35" name="tGlue" color="7" fill="4" visible="yes" active="yes"/>
+<layer number="36" name="bGlue" color="7" fill="5" visible="yes" active="yes"/>
+<layer number="37" name="tTest" color="7" fill="1" visible="yes" active="yes"/>
+<layer number="38" name="bTest" color="7" fill="1" visible="yes" active="yes"/>
+<layer number="39" name="tKeepout" color="4" fill="11" visible="yes" active="yes"/>
+<layer number="40" name="bKeepout" color="1" fill="11" visible="yes" active="yes"/>
+<layer number="41" name="tRestrict" color="4" fill="10" visible="yes" active="yes"/>
+<layer number="42" name="bRestrict" color="1" fill="10" visible="yes" active="yes"/>
+<layer number="43" name="vRestrict" color="2" fill="10" visible="yes" active="yes"/>
+<layer number="44" name="Drills" color="7" fill="1" visible="yes" active="yes"/>
+<layer number="45" name="Holes" color="7" fill="1" visible="yes" active="yes"/>
+<layer number="46" name="Milling" color="3" fill="1" visible="yes" active="yes"/>
+<layer number="47" name="Measures" color="7" fill="1" visible="yes" active="yes"/>
+<layer number="48" name="Document" color="7" fill="1" visible="yes" active="yes"/>
+<layer number="49" name="Reference" color="7" fill="1" visible="yes" active="yes"/>
 <layer number="50" name="dxf" color="7" fill="1" visible="no" active="no"/>
 <layer number="51" name="tDocu" color="7" fill="1" visible="yes" active="yes"/>
@@
 </autorouter>
 <elements>
-<element name="U$1" library="Module" package="ARDUINO-UNO" value="ARDUINO-UNO" x="0" y="0"/>
+<element name="U$1" library="Module" package="ARDUINO-UNO" value="" x="0" y="0"/>
 <element name="S1" library="Button" package="TS-DIP-4.5*4.5" value="" x="8.5725" y="39.37" rot="R180">
 <attribute name="MF" value="" x="8.5725" y="39.37" size="1.778" layer="27" rot="R180" display="off"/>
@@
 </element>
 <element name="LED4" library="Display" package="LED0805" value="RED" x="24.765" y="4.445" rot="R90"/>
-<element name="U$2" library="Senser" package="3362" value="33623362" x="33.02" y="10.16" rot="R180"/>
-<element name="U$3" library="Senser" package="BUZZER" value="BUZZER" x="40.005" y="42.545" rot="R90"/>
-<element name="U$4" library="Senser" package="DHT11" value="DHT11" x="24.13" y="41.275"/>
-<element name="U$5" library="Senser" package="TO92" value="LM35" x="48.895" y="8.255"/>
-<element name="U$6" library="Senser" package="LDR" value="LDR" x="40.005" y="8.89"/>
+<element name="U$2" library="Senser" package="3362" value="" x="33.02" y="10.16" rot="R180"/>
+<element name="U$3" library="Senser" package="BUZZER" value="" x="40.005" y="42.545" rot="R90"/>
+<element name="U$4" library="Senser" package="DHT11" value="" x="24.13" y="41.275"/>
+<element name="U$5" library="Senser" package="TO92" value="" x="48.895" y="8.255"/>
+<element name="U$6" library="Senser" package="LDR" value="" x="40.005" y="8.89"/>
 <element name="RELAY" library="Senser" package="RELAY-HK4100F-DC5V" value="" x="8.255" y="15.875"/>
 <element name="R1" library="RCLDA" package="R0805" value="331" x="5.08" y="50.8"/>
@@
 <element name="R4" library="RCLDA" package="R0805" value="471" x="22.225" y="4.445" rot="R270"/>
 <element name="R5" library="RCLDA" package="R0805" value="103" x="41.275" y="13.0175" rot="MR0"/>
-<element name="Q1" library="RCLDA" package="SOT23" value="S8050SOT23" x="10.795" y="15.875" rot="MR270"/>
-<element name="Q2" library="RCLDA" package="SOT23" value="S8050SOT23" x="37.465" y="42.545" rot="MR0"/>
+<element name="Q1" library="RCLDA" package="SOT23" value="" x="10.795" y="15.875" rot="MR270"/>
+<element name="Q2" library="RCLDA" package="SOT23" value="" x="37.465" y="42.545" rot="MR0"/>
 <element name="R6" library="RCLDA" package="R0805" value="103" x="8.5725" y="32.0675" rot="MR90"/>
 <element name="R7" library="RCLDA" package="R0805" value="222" x="14.9225" y="15.875" rot="MR90"/>
-<element name="D1" library="RCLDA" package="SMB" value="DIODESMB" x="5.715" y="15.875" rot="MR270"/>
+<element name="D1" library="RCLDA" package="SMB" value="" x="5.715" y="15.875" rot="MR270"/>
 <element name="R8" library="RCLDA" package="R0805" value="102" x="41.91" y="42.545" rot="MR270"/>
 <element name="R9" library="RCLDA" package="R0805" value="103" x="21.59" y="34.29" rot="MR180"/>
@@
 <element name="U$45" library="Logos" package="RED_050" value="" x="1.27" y="50.165"/>
 <element name="U$46" library="Logos" package="YELLOW_050" value="" x="1.27" y="47.625"/>
-<element name="U$8" library="Chip" package="SOP16" value="TM1650" x="57.15" y="15.875" rot="R180"/>
-<element name="S3" library="Button" package="TS-SMD_6*6_SHIELD" value="TS-SMD_6S6_SHIELD" x="6.35" y="4.445"/>
+<element name="U$8" library="Chip" package="SOP16" value="" x="57.15" y="15.875" rot="R180"/>
+<element name="S3" library="Button" package="TS-SMD_6*6_SHIELD" value="" x="6.35" y="4.445"/>
 <element name="R12" library="RCLDA" package="R0805" value="103" x="13.97" y="4.445" rot="R270"/>
 <element name="U$14" library="Logos" package="RESET_050" value="" x="4.1275" y="8.255"/>
@@
 <element name="U$25" library="Logos" package="D5_050" value="" x="31.115" y="24.765"/>
 <element name="U$32" library="Logos" package="D6_050" value="" x="31.115" y="27.94"/>
-<element name="U$15" library="Display" package="TN_AS_2_0.36INCH" value="3261AS" x="57.15" y="28.575"/>
+<element name="U$15" library="Display" package="TN_AS_2_0.36INCH" value="" x="57.15" y="28.575"/>
 <element name="U$39" library="Logos" package="MAKE_SOMETHING_FUN_050" value="" x="66.04" y="26.3525" rot="MR0"/>
 <element name="U$16" library="Logos" package="D4_050" value="" x="34.76625" y="33.02"/>
