File: projects/02 Arduino Basic Sensor Board/Arduino Basic Sensor Board.brd (EAGLE design)
At the start: 160 x 100 mm, 46 parts

Commit message: 2020.06.26.01
Parts:
- moved SV3 155.0 mm to (58.4, 7.62), turned to 270 degrees
- moved R5 147.8 mm to (41.9, 12.1), turned to 180 degrees
- moved SV5 145.5 mm to (43.8, 33.0), turned to 90 degrees
- moved SV4 135.2 mm to (41.3, 33.0), turned to 90 degrees
- moved R4 130.2 mm to (19.7, 3.81), turned to 270 degrees
- moved U$5 127.9 mm to (49.5, 6.99)
- moved S2 127.5 mm to (5.71, 41.3), turned to 90 degrees
- moved R15 124.1 mm to (59.7, 47.6), turned to 180 degrees
- moved SV1 117.3 mm to (38.7, 33.0), turned to 90 degrees
- moved LED4 117.2 mm to (22.2, 3.81), turned to 90 degrees
- moved LED3 116.9 mm to (55.2, 47.6), turned to 180 degrees
- moved U$6 115.8 mm to (40.6, 7.62)
- moved S1 113.1 mm to (5.71, 48.9)
- moved SV6 113.0 mm to (63.5, 42.5), turned to 90 degrees
- moved C1 107.1 mm to (17.1, 3.81), turned to 90 degrees
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Connections:
- removed net N$16: S2.3
- removed net N$17: S2.4
- net 5V0: now also S2.3
- net GND: now also S2.4
Routing:
- net D5: track 0.00 -> 57.2 mm
- net D6: track 0.00 -> 53.6 mm
- net 5V0: track 0.00 -> 46.0 mm
- net D11: track 0.00 -> 41.7 mm
- net D12: track 0.00 -> 37.6 mm
- net RESET: track 0.00 -> 35.8 mm
- net D13: track 0.00 -> 33.4 mm
- net N$8: track 0.00 -> 21.1 mm
- net N$32: track 0.00 -> 11.9 mm
- net TXD: track 0.00 -> 10.3 mm
- net RXD: track 0.00 -> 8.22 mm
- net N$9: track 0.00 -> 8.20 mm
- net D7: track 0.00 -> 7.99 mm
- net N$13: track 0.00 -> 6.98 mm
- net N$7: track 0.00 -> 3.02 mm
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- added copper zone on layer 1, net GND
- added copper zone on layer 16, net GND
Other:
- board outline removed
