File: projects/06 Emoji Board/Emoji Board.sch (EAGLE design)
At the start: 25 parts, among them M2 MAX7219, U2 ATMEGA8A-AU-TQFP32, Y1 16MHZ

Commit message: 2020.06.24.04
Parts:
- removed C5: 104, RCLDA:C0805
- removed CT1: 100UF, RCLDA:ALUMINUM-SMD-100UF-50V(D6.0-H6.0MM)
- removed D1: DIODESMB, RCLDA:DIODESMB
- removed FUSE: 1.1A, RCLDA:FUSE0805
- removed LED1: RED, Display:LEDCHIPLED_0805
- removed R1: 471, RCLDA:R0805
- removed S1: (no value), Button:TS-DIP-4.54.5
- removed SJ1: (no value), Jumper:SJ
- removed U1: (no value), Chip:MCU-ATMEGA328P-PU(DIP28)
- removed X1: (no value), Connector:AK500/2
- added G1, G3: CR1220, Power:CR1220
- added U$1: TS-DIP, Button:TS-DIP
- added U$2: AMS1117-5V0SOT22, Chip:AMS1117-5V0SOT22
Connections:
- removed net AREF: SJ1.1, U1.AREF
- removed net N$4: LED1.A, R1.1
- removed net SCL: U1.PC5
- removed net SDA: U1.PC4
- new net A4: U2.PC4(ADC4/SDA)
- new net A5: U2.PC5(ADC5/SCL)
- new net A6: U2.ADC6
- new net A7: U2.ADC7
- new net N$8: U2.AREF
- new net N$9: U2.AVCC
- net +5V: now also U$2.OUT, U2.VCC@1, U2.VCC@2; no longer D1.1, R1.2, SJ1.2, U1.AVCC, U1.VCC
- net A0: now also U2.PC0(ADC0); no longer U1.PC0
- net A1: now also U2.PC1(ADC1); no longer U1.PC1
- net A2: now also U2.PC2(ADC2); no longer U1.PC2
- net A3: now also U2.PC3(ADC3); no longer U1.PC3
- net D2: now also U2.PD2(INT0); no longer U1.PD2
- net D3: now also U2.PD3(INT1); no longer U1.PD3
- net D4: now also U2.PD4(XCK/T0); no longer U1.PD4
- net D5: now also U2.PD5(T1); no longer U1.PD5
- net D6: now also U2.PD6(AIN0); no longer U1.PD6
- net D7: now also U2.PD7(AIN1); no longer U1.PD7
- net D8: now also U2.PB0(ICP); no longer U1.PB0
- net D9: now also U2.PB1(OC1A); no longer U1.PB1
- net GND: now also G1.-, U$1.P, U$2.GND, U2.GND, U2.GND@1, U2.GND@2; no longer C5.2, CT1.-, LED1.C, S1.P, S1.P1, U1.GND@1, U1.GND@2, X1-1.KL
- net MISO: now also U2.PB4(MISO); no longer U1.PB4
- net MOSI: now also U2.PB3(MOSI/OC2); no longer U1.PB3
- net N$2: now also G1.+, G3.-; no longer D1.2, FUSE.P$2
- net RST: now also U$1.S, U2.PC6(/RESET); no longer S1.S, S1.S1, U1.!RST
- net RXD: now also U2.PD0(RXD); no longer U1.PD0/RX
- net SCK: now also U2.PB5(SCK); no longer U1.PB5
- net SS: now also U2.PB2(SS/OC1B); no longer U1.PB2
- net TXD: now also U2.PD1(TXD); no longer U1.PD1/TX
- net VCC: now also G3.+, U$2.VIN; no longer C5.1, CT1.+, FUSE.P$1, X1-2.KL
- net X1: now also U2.PB6(XTAL1/TOSC1); no longer U1.X1
- net X2: now also U2.PB7(XTAL2/TOSC2); no longer U1.X2
Other:
- moved on the sheet: C1, C6, LED2, R2, R3, SV1, U2

Commit message: 2020.06.27.01
Parts:
- removed C6: 104, RCLDA:C0805
- removed G3: CR1220, Power:CR1220
- removed LED2: GREEN, Display:LEDCHIPLED_0805
- removed LED3: YELLOW, Display:LEDCHIPLED_0805
- removed R6: R0805, RCLDA:R0805
- removed U2: ATMEGA8A-AU-TQFP32, Chip:ATMEGA8A-AU
- removed Y1: 16MHZ, Crystal:DIP-CRYSTAL-16MHZ-18PF-30PPM-40R(HC49US)
- added C2: C0805, RCLDA:C0805
- added G2: CR1220, Power:CR1220
- added LED1, LED4: (no value), Display:LEDSML0805
- added R1: 103, RCLDA:R0805
- added SV2: (no value), Pin-Header:MA06-1
- added U$10, U$11, U$4, U$5, U$6, U$7, U$8, U$9: CONNECTOR, Connector:CONNECTOR
- added U1: ATMEGA8A-AU-TQFP32, Chip:ATMEGA8A-AU
- added Y2: 16MHZ, Crystal:DIP-CRYSTAL-16MHZ-18PF-30PPM-40R(HC49US)
- C3, C4: value 22p -> C0805
- R2: value 103 -> R0805
- R3, R4: value 471 -> R0805
- SV1: device Pin-Header:MA06-1 -> Pin-Header:MA04-1
- renumbered L2 to U$3, M2 to U$12
Connections:
- removed net D7: U2.PD7(AIN1)
- removed net D8: U2.PB0(ICP)
- removed net D9: U2.PB1(OC1A)
- removed net N$3: C1.2, SV1.6
- net +5V: now also C1.2, C4.2, R1.1, R3.1, R4.1, SV1.4, SV2.6, U1.VCC@1, U1.VCC@2; no longer C6.2, R2.1, R3.2, R6.1, SV1.3, U2.VCC@1, U2.VCC@2
- net A0: now also U1.PC0(ADC0); no longer U2.PC0(ADC0)
- net A1: now also U1.PC1(ADC1); no longer U2.PC1(ADC1)
- net A2: now also U1.PC2(ADC2); no longer U2.PC2(ADC2)
- net A3: now also U1.PC3(ADC3); no longer U2.PC3(ADC3)
- net A4: now also U1.PC4(ADC4/SDA); no longer U2.PC4(ADC4/SDA)
- net A5: now also U1.PC5(ADC5/SCL); no longer U2.PC5(ADC5/SCL)
- net A6: now also U1.ADC6; no longer U2.ADC6
- net A7: now also U1.ADC7; no longer U2.ADC7
- net CLK: now also U1.PB0(ICP)
- net CS: now also U1.PB1(OC1A)
- net D2: now also U1.PD2(INT0); no longer U2.PD2(INT0)
- net D3: now also U1.PD3(INT1); no longer U2.PD3(INT1)
- net D4: now also U1.PD4(XCK/T0); no longer U2.PD4(XCK/T0)
- net D5: now also U1.PD5(T1); no longer U2.PD5(T1)
- net D6: now also U1.PD6(AIN0); no longer U2.PD6(AIN0)
- net DIN: now also U1.PD7(AIN1)
- net GND: now also C2.1, G2.-, LED1.C, LED4.C, SV2.1, U1.GND, U1.GND@1, U1.GND@2; no longer C6.1, G1.-, LED2.C, LED3.C, SV1.2, U2.GND, U2.GND@1, U2.GND@2
- net MISO: now also SV2.4, U1.PB4(MISO); no longer U2.PB4(MISO)
- net MOSI: now also SV2.3, U1.PB3(MOSI/OC2); no longer U2.PB3(MOSI/OC2)
- net N$1: now also LED4.A, R2.2; no longer LED3.A, R4.1
- net N$10: now also LED1.A, R3.2; no longer LED2.A, R3.1
- net N$2: now also G1.-, G2.+; no longer G1.+, G3.-
- net N$6: now also R4.2; no longer R6.2
- net N$8: now also U1.AREF; no longer U2.AREF
- net N$9: now also U1.AVCC; no longer U2.AVCC
- net RST: now also R1.2, U1.PC6(/RESET); no longer R2.2, U2.PC6(/RESET)
- net RXD: now also SV1.2, U1.PD0(RXD); no longer SV1.4, U2.PD0(RXD)
- net SCK: now also R2.1, SV2.5, U1.PB5(SCK); no longer R4.2, U2.PB5(SCK)
- net SS: now also SV2.2, U1.PB2(SS/OC1B); no longer U2.PB2(SS/OC1B)
- net TXD: now also SV1.3, U1.PD1(TXD); no longer SV1.5, U2.PD1(TXD)
- net VCC: now also G1.+; no longer G3.+
- net X1: now also C2.2, U1.PB6(XTAL1/TOSC1), Y2.2; no longer C3.2, U2.PB6(XTAL1/TOSC1), Y1.2
- net X2: now also C3.2, U1.PB7(XTAL2/TOSC2), Y2.1; no longer C4.2, U2.PB7(XTAL2/TOSC2), Y1.1
Other:
- moved on the sheet: C1, C3, C4, G1, R2, R3, R4, U$1
