File: exercise/demo/untitled.sch (EAGLE design)
At the start: 19 parts

Commit message: 2020.07.15.01
Parts:
- removed LED1, LED10, LED11, LED12, LED13, LED14, LED15, LED16, LED2, LED3, LED4, LED5, LED6, LED7, LED8, LED9: (no value), Display:LED
- removed U$2: 3621AS, Display:3621AS
- added R1: R0805, RCLDA:R0805
- U$1: value TM1650 -> DHT11; device Chip:TM1650 -> Senser:DHT11
Connections:
- removed net A: LED1.A, LED9.C, U$1.A, U$2.A
- removed net B: LED10.C, LED2.A, U$1.B, U$2.B
- removed net C: LED11.C, LED3.A, U$1.C, U$2.C
- removed net D: LED12.C, LED4.A, U$1.D, U$2.D
- removed net DIG1: LED1.C, LED2.C, LED3.C, LED4.C, LED5.C, LED6.C, LED7.C, LED8.C, U$1.DIG1, U$2.DIG1
- removed net DIG2: LED10.A, LED11.A, LED12.A, LED13.A, LED14.A, LED15.A, LED16.A, LED9.A, U$1.DIG2, U$2.DIG2
- removed net E: LED13.C, LED5.A, U$1.E, U$2.E
- removed net F: LED14.C, LED6.A, U$1.F, U$2.F
- removed net G: LED15.C, LED7.A, U$1.G, U$2.G
- removed net H: LED16.C, LED8.A, U$1.H, U$2.DP
- removed net SCL: ARDUINO-UNO.A5/SCL, U$1.SCL
- removed net SDA: ARDUINO-UNO.A4/SDA, U$1.SDA
- new net N$1: ARDUINO-UNO.D7, R1.1, U$1.DAT
- net 5V0: now also R1.2, U$1.VCC; no longer U$1.VDD

Commit message: 2020.07.15.02
Connections:
- net N$1: now also ARDUINO-UNO.D8; no longer ARDUINO-UNO.D7
Other:
- moved on the sheet: R1, U$1
Changed lines of the file:
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@@
 <setting verticaltext="up"/>
 </settings>
-<grid distance="50" unitdist="mil" unit="mil" style="lines" multiple="1" display="yes" altdistance="25" altunitdist="mil" altunit="mil"/>
+<grid distance="50" unitdist="mil" unit="mil" style="lines" multiple="1" display="no" altdistance="25" altunitdist="mil" altunit="mil"/>
 <layers>
 <layer number="1" name="Top" color="4" fill="1" visible="no" active="no"/>
@@
 <instance part="FRAME1" gate="G$1" x="0" y="0"/>
 <instance part="ARDUINO-UNO" gate="G$1" x="66.04" y="121.92"/>
-<instance part="U$1" gate="G$1" x="107.95" y="118.11" rot="R270"/>
-<instance part="R1" gate="G$1" x="87.63" y="127" rot="R90"/>
+<instance part="U$1" gate="G$1" x="107.95" y="120.65" rot="R270"/>
+<instance part="R1" gate="G$1" x="87.63" y="129.54" rot="R90"/>
 </instances>
 <busses>
@@
 <wire x1="41.91" y1="148.59" x2="87.63" y2="148.59" width="0.1524" layer="91"/>
 <wire x1="87.63" y1="148.59" x2="92.71" y2="148.59" width="0.1524" layer="91"/>
-<wire x1="92.71" y1="148.59" x2="92.71" y2="121.92" width="0.1524" layer="91"/>
+<wire x1="92.71" y1="148.59" x2="92.71" y2="124.46" width="0.1524" layer="91"/>
 <pinref part="U$1" gate="G$1" pin="VCC"/>
-<wire x1="92.71" y1="121.92" x2="95.25" y2="121.92" width="0.1524" layer="91"/>
+<wire x1="92.71" y1="124.46" x2="95.25" y2="124.46" width="0.1524" layer="91"/>
 <pinref part="R1" gate="G$1" pin="2"/>
-<wire x1="87.63" y1="132.08" x2="87.63" y2="148.59" width="0.1524" layer="91"/>
+<wire x1="87.63" y1="134.62" x2="87.63" y2="148.59" width="0.1524" layer="91"/>
 <junction x="87.63" y="148.59"/>
 </segment>
@@
 <wire x1="41.91" y1="119.38" x2="48.26" y2="119.38" width="0.1524" layer="91"/>
 <pinref part="U$1" gate="G$1" pin="GND"/>
-<wire x1="95.25" y1="114.3" x2="92.71" y2="114.3" width="0.1524" layer="91"/>
-<wire x1="92.71" y1="114.3" x2="92.71" y2="95.25" width="0.1524" layer="91"/>
+<wire x1="95.25" y1="116.84" x2="92.71" y2="116.84" width="0.1524" layer="91"/>
+<wire x1="92.71" y1="116.84" x2="92.71" y2="95.25" width="0.1524" layer="91"/>
 <wire x1="92.71" y1="95.25" x2="41.91" y2="95.25" width="0.1524" layer="91"/>
 <wire x1="41.91" y1="95.25" x2="41.91" y2="119.38" width="0.1524" layer="91"/>
@@
 <net name="N$1" class="0">
 <segment>
-<pinref part="ARDUINO-UNO" gate="G$1" pin="D7"/>
 <pinref part="U$1" gate="G$1" pin="DAT"/>
-<wire x1="83.82" y1="119.38" x2="87.63" y2="119.38" width="0.1524" layer="91"/>
 <pinref part="R1" gate="G$1" pin="1"/>
-<wire x1="87.63" y1="119.38" x2="95.25" y2="119.38" width="0.1524" layer="91"/>
-<wire x1="87.63" y1="119.38" x2="87.63" y2="121.92" width="0.1524" layer="91"/>
-<junction x="87.63" y="119.38"/>
+<wire x1="87.63" y1="121.92" x2="95.25" y2="121.92" width="0.1524" layer="91"/>
+<wire x1="87.63" y1="121.92" x2="87.63" y2="124.46" width="0.1524" layer="91"/>
+<pinref part="ARDUINO-UNO" gate="G$1" pin="D8"/>
+<wire x1="83.82" y1="121.92" x2="87.63" y2="121.92" width="0.1524" layer="91"/>
+<junction x="87.63" y="121.92"/>
 </segment>
 </net>
